File: hard/led_alive.kicad_sch (KiCad schematic)
At the start: 0 parts

Commit message: edit
Parts:
- added D8: LED, symbol Device:LED
- added R9: R, symbol Device:R
Connections:
- new net: D8.2 (A), R9.2
- new net GND: D8.1 (K)
- new net LED_ALIVE: R9.1
