File: hard/temperature_sensor.kicad_sch (KiCad schematic)
At the start: 0 parts

Commit message: edit
Parts:
- added C10, C11: C, symbol Device:C
- added R10: R, symbol Device:R
- added U2: MCP9700Ax-ETT, Package_TO_SOT_SMD:SOT-23, symbol Sensor_Temperature:MCP9700Ax-ETT
Connections:
- new net: R10.1, U2.2 (V_{OUT})
- new net GND: C10.2, C11.2, U2.3 (GND)
- new net TEMP: C10.1, R10.2
- new net VDD: C11.1, U2.1 (V_{DD})
