File: hard/accelerometer.kicad_sch (KiCad schematic)
At the start: 0 parts

Commit message: update
Parts:
- added C27, C28: C, symbol Device:C
- added R14, R15: R, symbol Device:R
Connections:
- new net +3V3: C27.1, R14.1, R15.1
- new net ACC_SCL: R15.2
- new net ACC_SDA: R14.2
- new net GND: C27.2, C28.2
