File: hard/display_buttons.kicad_sch (KiCad schematic)
At the start: 0 parts

Commit message: edit
Parts:
- added C4, C5, C6, C7: C, symbol Device:C
- added R5, R6, R7, R8: R, symbol Device:R
- added SW2, SW3, SW4, SW5: SW_MEC_5G, symbol Switch:SW_MEC_5G
Connections:
- new net GND: C4.2, C5.2, C6.2, C7.2, SW2.3 (B), SW2.4 (B), SW3.3 (B), SW3.4 (B), SW4.3 (B), SW4.4 (B), SW5.3 (B), SW5.4 (B)
- new net SW_DOWN: C4.1, C5.1, C6.1, C7.1, R5.2, R6.2, R7.2, R8.2, SW2.1 (A), SW2.2 (A), SW3.1 (A), SW3.2 (A), SW4.1 (A), SW4.2 (A), SW5.1 (A), SW5.2 (A)
- new net VDD: R5.1, R6.1, R7.1, R8.1

Commit message: update
Other:
- moved on the sheet: C4, C5, C6, C7, R5, R6, R7, R8, SW2, SW3, SW4, SW5
