File: hard/gps.kicad_sch (KiCad schematic)
At the start: 0 parts

Commit message: update
Parts:
- added C12, C13: C, symbol Device:C
- added Q3: Q_NMOS_SGD, symbol Transistor_FET:Q_NMOS_SGD
- added R11: R, symbol Device:R
- added U3: SAM-M8Q, RF_GPS:ublox_SAM-M8Q, symbol RF_GPS:SAM-M8Q
Connections:
- new net: C12.1, C13.1, Q3.1 (S), U3.17 (VCC), U3.2 (VCC_IO), U3.3 (V_BCKP)
- new net GND: C12.2, C13.2, U3.1 (GND), U3.10 (GND), U3.11 (GND), U3.15 (GND), U3.16 (GND), U3.20 (GND), U3.4 (GND), U3.5 (GND), U3.6 (GND)
- new net RX_SAM: U3.14 (RXD)
- new net SAM_EN: Q3.2 (G), R11.2
- new net SAM_PPS: U3.7 (TIMEPULSE)
- new net SAM_RST: U3.18 (~{RESET})
- new net TX_SAM: U3.13 (TXD)
- new net VDD: Q3.3 (D), R11.1
- no-connect marks 0 -> 4
