File: hard/lvr.kicad_sch (KiCad schematic)
At the start: 9 parts

Commit message: edit
Parts:
- added U501: SC662K-3-3V, Package_TO_SOT_SMD:SOT-23, symbol Regulator_Linear:AP2127N-1.0
Connections:
- net +3V3: now also U501.2 (VO); no longer C504.1
- new net +5V: C504.1, U501.3 (VI)
Other:
- moved on the sheet: C505, C512
Changed lines of the file:
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@@
+	)
+	(junction
+		(at 128.27 85.09)
+		(diameter 0)
+		(color 0 0 0 0)
 	)
 	(junction
@@
 	)
 	(junction
-		(at 121.92 85.09)
+		(at 116.84 85.09)
 		(diameter 0)
 		(color 0 0 0 0)
 	)
-	(junction
-		(at 105.41 85.09)
-		(diameter 0)
-		(color 0 0 0 0)
-	)
 	(wire
 		(pts
@@
 	(wire
 		(pts
-			(xy 87.63 85.09) (xy 105.41 85.09)
+			(xy 87.63 85.09) (xy 99.06 85.09)
 		)
 		(stroke
@@
 	(wire
 		(pts
+			(xy 114.3 85.09) (xy 116.84 85.09)
+		)
+		(stroke
+			(width 0)
+			(type default)
+		)
+	)
+	(wire
+		(pts
 			(xy 177.8 92.71) (xy 182.88 92.71)
 		)
@@
 	(wire
 		(pts
-			(xy 130.81 85.09) (xy 121.92 85.09)
+			(xy 130.81 85.09) (xy 128.27 85.09)
 		)
 		(stroke
@@
 	(wire
 		(pts
-			(xy 105.41 92.71) (xy 105.41 96.52)
+			(xy 116.84 85.09) (xy 128.27 85.09)
+		)
+		(stroke
+			(width 0)
+			(type default)
+		)
+	)
+	(wire
+		(pts
+			(xy 116.84 92.71) (xy 116.84 96.52)
 		)
 		(stroke
@@
 	(wire
 		(pts
-			(xy 105.41 85.09) (xy 121.92 85.09)
-		)
-		(stroke
-			(width 0)
-			(type default)
-		)
-	)
-	(wire
-		(pts
 			(xy 143.51 102.87) (xy 151.13 102.87)
 		)
@@
 	(wire
 		(pts
-			(xy 121.92 92.71) (xy 121.92 96.52)
+			(xy 128.27 92.71) (xy 128.27 96.52)
 		)
 		(stroke
@@
 		(length 2.54)
 		(shape round)
-		(at 96.52 85.09 0)
+		(at 91.44 85.09 0)
 		(effects
 			(font
@@
 		)
 		(property "Netclass" "TP502"
-			(at 97.282 81.026 0)
+			(at 92.202 81.026 0)
 			(effects
 				(font
@@
 		)
 		(property "Component Class" "5V"
-			(at 98.044 83.058 0)
+			(at 92.964 83.058 0)
 			(effects
 				(font
@@
 	(symbol
 		(lib_id "Device:C")
-		(at 105.41 88.9 0)
+		(at 116.84 88.9 0)
 		(unit 1)
 		(exclude_from_sim no)
@@
 		(dnp no)
 		(property "Reference" "C512"
-			(at 107.95 89.408 0)
+			(at 119.38 89.408 0)
 			(effects
 				(font
@@
 		)
 		(property "Value" "100n"
-			(at 107.95 91.948 0)
+			(at 119.38 91.948 0)
 			(effects
 				(font
@@
 		)
 		(property "Footprint" ""
-			(at 106.3752 92.71 0)
+			(at 117.8052 92.71 0)
 			(effects
 				(font
@@
 		)
 		(property "Datasheet" "~"
-			(at 105.41 88.9 0)
+			(at 116.84 88.9 0)
 			(effects
 				(font
@@
 		)
 		(property "Description" "Unpolarized capacitor"
-			(at 105.41 88.9 0)
+			(at 116.84 88.9 0)
 			(effects
 				(font
@@
 	(symbol
 		(lib_id "power:GND")
-		(at 121.92 96.52 0)
+		(at 128.27 96.52 0)
 		(unit 1)
 		(exclude_from_sim no)
@@
 		(fields_autoplaced yes)
 		(property "Reference" "#PWR011"
-			(at 121.92 102.87 0)
+			(at 128.27 102.87 0)
 			(effects
 				(font
@@
 		)
 		(property "Value" "GND"
-			(at 121.92 101.6 0)
-			(effects
-				(font
-					(size 1.27 1.27)
-				)
-			)
-		)
-		(property "Footprint" ""
-			(at 121.92 96.52 0)
+			(at 128.27 101.6 0)
+			(effects
+				(font
+					(size 1.27 1.27)
+				)
+			)
+		)
+		(property "Footprint" ""
+			(at 128.27 96.52 0)
 			(effects
 				(font
@@
 		)
 		(property "Datasheet" ""
-			(at 121.92 96.52 0)
+			(at 128.27 96.52 0)
 			(effects
 				(font
@@
 		)
 		(property "Description" "Power symbol creates a global label with name \"GND\" , ground"
-			(at 121.92 96.52 0)
+			(at 128.27 96.52 0)
 			(effects
 				(font
@@
 	)
 	(symbol
+		(lib_id "Regulator_Linear:AP2127N-1.0")
+		(at 106.68 85.09 0)
+		(unit 1)
+		(exclude_from_sim no)
+		(in_bom yes)
+		(on_board yes)
+		(dnp no)
+		(fields_autoplaced yes)
+		(property "Reference" "U501"
+			(at 106.68 78.74 0)
+			(effects
+				(font
+					(size 1.27 1.27)
+				)
+			)
+		)
+		(property "Value" "SC662K-3-3V"
+			(at 106.68 81.28 0)
+			(effects
+				(font
+					(size 1.27 1.27)
+				)
+			)
+		)
+		(property "Footprint" "Package_TO_SOT_SMD:SOT-23"
+			(at 106.68 79.375 0)
+			(effects
+				(font
+					(size 1.27 1.27)
+					(italic yes)
+				)
+				(hide yes)
+			)
+		)
+		(property "Datasheet" "https://www.diodes.com/assets/Datasheets/AP2127.pdf"
+			(at 106.68 85.09 0)
+			(effects
+				(font
+					(size 1.27 1.27)
+				)
+				(hide yes)
+			)
+		)
+		(property "Description" "300mA low dropout linear regulator, shutdown pin, 2.5V-6V input voltage, 1.0V fixed positive output, SOT-23 package"
+			(at 106.68 85.09 0)
+			(effects
+				(font
+					(size 1.27 1.27)
+				)
+				(hide yes)
+			)
+		)
+		(pin "3"
+		)
+		(pin "2"
+		)
+		(pin "1"
+		)
+		(instances
+			(project ""
+				(path "/13844229-b559-4868-a710-53f590233cb2/ca9a428d-b29f-459a-8b79-10121d41243b/5caab3ad-a795-4284-8cea-618258e8e471"
+					(reference "U501")
+					(unit 1)
+				)
+			)
+		)
+	)
+	(symbol
 		(lib_id "Device:NetTie_2")
 		(at 153.67 102.87 0)
@@
 	(symbol
 		(lib_id "power:GND")
-		(at 105.41 96.52 0)
+		(at 116.84 96.52 0)
 		(unit 1)
 		(exclude_from_sim no)
@@
 		(fields_autoplaced yes)
 		(property "Reference" "#PWR09"
-			(at 105.41 102.87 0)
+			(at 116.84 102.87 0)
 			(effects
 				(font
@@
 		)
 		(property "Value" "GND"
-			(at 105.41 101.6 0)
-			(effects
-				(font
-					(size 1.27 1.27)
-				)
-			)
-		)
-		(property "Footprint" ""
-			(at 105.41 96.52 0)
+			(at 116.84 101.6 0)
+			(effects
+				(font
+					(size 1.27 1.27)
+				)
+			)
+		)
+		(property "Footprint" ""
+			(at 116.84 96.52 0)
 			(effects
 				(font
@@
 		)
 		(property "Datasheet" ""
-			(at 105.41 96.52 0)
+			(at 116.84 96.52 0)
 			(effects
 				(font
@@
 		)
 		(property "Description" "Power symbol creates a global label with name \"GND\" , ground"
-			(at 105.41 96.52 0)
+			(at 116.84 96.52 0)
 			(effects
 				(font
@@
 	(symbol
 		(lib_id "Device:C")
-		(at 121.92 88.9 0)
+		(at 128.27 88.9 0)
 		(unit 1)
 		(exclude_from_sim no)
@@
 		(dnp no)
 		(property "Reference" "C505"
-			(at 125.222 88.646 0)
+			(at 131.572 88.646 0)
 			(effects
 				(font
@@
 		)
 		(property "Value" "1u"
-			(at 125.476 90.678 0)
+			(at 131.826 90.678 0)
 			(effects
 				(font
@@
 		)
 		(property "Footprint" ""
-			(at 122.8852 92.71 0)
+			(at 129.2352 92.71 0)
 			(effects
 				(font
@@
 		)
 		(property "Datasheet" "~"
-			(at 121.92 88.9 0)
+			(at 128.27 88.9 0)
 			(effects
 				(font
@@
 		)
 		(property "Description" "Unpolarized capacitor"
-			(at 121.92 88.9 0)
-			(effects
-				(font
+			(at 128.27 88.9 0)
+			(effects
+				(font

Commit message: update
Parts:
- removed C505: 1u, symbol Device:C
- removed U501: SC662K-3-3V, Package_TO_SOT_SMD:SOT-23, symbol Regulator_Linear:AP2127N-1.0
- added U5: XC6705A331MR-G, Package_TO_SOT_SMD:SOT-23-5, symbol Regulator_Linear:XC6210B332MR
Connections:
- net +3V3: now also U5.5 (VOUT)
- net +5V: now also U5.1 (VIN), U5.3 (CE)
- net GND: now also U5.2 (GND)
Other:
- moved on the sheet: C504
