File: hard/mini_usb.kicad_sch (KiCad schematic)
At the start: 8 parts, among them J502 USB_B_Mini, Q501 IRLML9301

Commit message: update
Other:
- moved on the sheet: D503, FB501, J502, Q501, R501, R502, R503, R504
