File: hard/sensors.kicad_sch (KiCad schematic)
At the start: 0 parts

Commit message: update
Parts:
- added C29, C30, C31, C32, C33, C34: C, symbol Device:C
- added Q4: Q_NMOS_SGD, symbol Transistor_FET:Q_NMOS_SGD
- added R16, R17, R18, R19: R, symbol Device:R
- added U6: MCP9700Ax-ETT, Package_TO_SOT_SMD:SOT-23, symbol Sensor_Temperature:MCP9700Ax-ETT
- added U7: SAM-M8Q, RF_GPS:ublox_SAM-M8Q, symbol RF_GPS:SAM-M8Q
Connections:
- new net: R18.1, U6.2 (V_{OUT})
- new net: C33.1, C34.1, Q4.1 (S), U7.17 (VCC), U7.2 (VCC_IO), U7.3 (V_BCKP)
- new net +3V3: C29.1, R16.1, R17.1
- new net ACC_SCL: R17.2
- new net ACC_SDA: R16.2
- new net GND: C29.2, C30.2, C31.2, C32.2, C33.2, C34.2, U6.3 (GND), U7.1 (GND), U7.10 (GND), U7.11 (GND), U7.15 (GND), U7.16 (GND), U7.20 (GND), U7.4 (GND), U7.5 (GND), U7.6 (GND)
- new net RX_SAM: U7.14 (RXD)
- new net SAM_EN: Q4.2 (G), R19.2
- new net SAM_PPS: U7.7 (TIMEPULSE)
- new net SAM_RST: U7.18 (~{RESET})
- new net TEMP: C32.1, R18.2
- new net TX_SAM: U7.13 (TXD)
- new net VDD: C31.1, Q4.3 (D), R19.1, U6.1 (V_{DD})
- no-connect marks 0 -> 4
Other:
- removed sheet accelerometer
- removed sheet esp
- removed sheet expansions
- removed sheet gps
- removed sheet temperature_sensor

Commit message: update
Parts:
- added C45: 4.7u, symbol Device:C
- added C47: C, symbol Device:C
- added J10: SERVO_3, symbol Connector:Conn_01x03_Pin
- added J6: I2C_3V3, symbol Connector:Conn_01x04_Pin
- added J7: UART0_3V3, symbol Connector:Conn_01x04_Pin
- added J8: SERVO_1, symbol Connector:Conn_01x03_Pin
- added J9: SERVO_2, symbol Connector:Conn_01x03_Pin
- added R27: 10k, symbol Device:R
- added U8: MMA8451Q, Package_DFN_QFN:DFN-10_2x2mm_P0.4mm, symbol Sensor_Motion:MMA8653FCR1
- added U9: ESP-01, RF_Module:ESP-07, symbol RF_Module:ESP-07
- C41: renamed from C29; value C -> 100n
- C42: renamed from C33; value C -> 4u7
- C43: renamed from C30; value C -> 100n
- C44: renamed from C34; value C -> 100n
- C46: renamed from C31; value C -> 100n
- C48: renamed from C32; value C -> 1u 6V3
- Q3: renamed from Q4; value Q_NMOS_SGD -> IRLML9301
- R24: renamed from R19; value R -> 10k
- R25: renamed from R16; value R -> 4.7k
- R26: renamed from R17; value R -> 4.7k
- R28: renamed from R18; value R -> 470
- U10: renamed from U6; value MCP9700Ax-ETT -> TC1047A
Connections:
- net +3V3: now also C45.1, C47.1, J6.4 (Pin_4), J7.4 (Pin_4), R27.1, U8.1 (VDDIO), U8.14 (VDD), U9.5 (VCC)
- net ACC_INT1: now also U8.11 (INT1)
- net ACC_INT2: now also U8.9 (INT2)
- net ACC_SCL: now also U8.4 (SCL)
- net ACC_SDA: now also U8.6 (SDA)
- net ESP_EN: now also U9.7 (EN)
- net ESP_RX: now also U9.4 (UART_RX)
- net ESP_TX: now also U9.8 (UART_TX)
- net EXT_I2C_SCL: now also J6.3 (Pin_3)
- net EXT_I2C_SDA: now also J6.2 (Pin_2)
- net GND: now also C45.2, C47.2, J10.3 (Pin_1), J6.1 (Pin_1), J7.1 (Pin_1), J8.3 (Pin_1), J9.3 (Pin_1), U8.10 (GND), U8.12 (GND), U8.5 (GND), U8.7 (SAO), U9.1 (GND); no longer U7.10 (GND), U7.11 (GND), U7.15 (GND), U7.16 (GND), U7.20 (GND), U7.4 (GND), U7.5 (GND), U7.6 (GND)
- net RX_SAM: now also J7.2 (Pin_2)
- net SERVO_1: now also J8.1 (Pin_3)
- net SERVO_2: now also J9.1 (Pin_3)
- net SERVO_3: now also J10.1 (Pin_3)
- net VDD: no longer C46.1, U10.1 (V_{DD})
- net at C43.1: now also U8.2 (BYP)
- new net: R27.2, U9.6 (~{RST})
- new net +3.3VA: C46.1, U10.1 (V_{DD})
- new net +5V: J10.2 (Pin_2), J8.2 (Pin_2), J9.2 (Pin_2)
- new net UART_RX: J7.3 (Pin_3)
- no-connect marks 4 -> 11
Other:
- note added: "Accelerometro"
- note added: "Espansioni"
- note added: "Modulo GPS SAM-M8Q"
- note added: "Sensore Temperatura"
- moved on the sheet: C41, C42, C43, C44, C46, C48, Q3, R24, R25, R26, R28, U10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
