File: hard/sensors.kicad_sch (KiCad schematic)
At the start: 23 parts, among them J10 SERVO_3, J6 I2C_3V3, J7 UART0_3V3, J8 SERVO_1, J9 SERVO_2, Q3 IRLML9301, U10 TC1047A, U7 SAM-M8Q, U8 MMA8451Q, U9 ESP-01

Commit message: update
Parts:
- removed Q3: IRLML9301, Package_TO_SOT_SMD:SOT-23, symbol Transistor_FET:Q_NMOS_SGD
- added Q3: IRLML9301, Package_TO_SOT_SMD:SOT-23, symbol Transistor_FET:IRLML9301
Connections:
- net VDD is gone; now on net +3V3: R24.1
- net +3V3: now also Q3.2 (S)
- net GND: no longer U7.10 (GND), U7.11 (GND), U7.15 (GND), U7.16 (GND), U7.20 (GND), U7.4 (GND), U7.5 (GND), U7.6 (GND)
- net SAM_EN: now also Q3.1 (G)
- net at C42.1, C44.1, U7.17 (VCC)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: now also Q3.3 (D)
Changed lines of the file:
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@@
 	)
 	(junction
+		(at 45.72 95.25)
+		(diameter 0)
+		(color 0 0 0 0)
+	)
+	(junction
 		(at 49.53 53.34)
 		(diameter 0)
@@
 	)
 	(junction
-		(at 45.72 95.25)
+		(at 57.15 87.63)
 		(diameter 0)
 		(color 0 0 0 0)
@@
 	)
 	(junction
-		(at 57.15 87.63)
+		(at 81.28 87.63)
 		(diameter 0)
 		(color 0 0 0 0)
@@
 	)
 	(junction
-		(at 82.55 100.33)
-		(diameter 0)
-		(color 0 0 0 0)
-	)
-	(junction
 		(at 31.75 67.31)
 		(diameter 0)
@@
 	(wire
 		(pts
-			(xy 82.55 100.33) (xy 82.55 87.63)
+			(xy 85.09 100.33) (xy 85.09 87.63)
 		)
 		(stroke
@@
 	(wire
 		(pts
+			(xy 50.8 87.63) (xy 57.15 87.63)
+		)
+		(stroke
+			(width 0)
+			(type default)
+		)
+	)
+	(wire
+		(pts
 			(xy 19.05 85.09) (xy 19.05 87.63)
 		)
@@
 	(wire
 		(pts
-			(xy 85.09 104.14) (xy 85.09 100.33)
-		)
-		(stroke
-			(width 0)
-			(type default)
-		)
-	)
-	(wire
-		(pts
 			(xy 19.05 87.63) (xy 22.86 87.63)
 		)
@@
 	(wire
 		(pts
-			(xy 44.45 176.53) (xy 50.8 176.53)
+			(xy 81.28 87.63) (xy 69.85 87.63)
 		)
 		(stroke
@@
 	(wire
 		(pts
-			(xy 22.86 87.63) (xy 40.64 87.63)
+			(xy 44.45 176.53) (xy 50.8 176.53)
 		)
 		(stroke
@@
 	(wire
 		(pts
-			(xy 50.8 87.63) (xy 57.15 87.63)
+			(xy 22.86 87.63) (xy 40.64 87.63)
 		)
 		(stroke
@@
 	(wire
 		(pts
+			(xy 85.09 100.33) (xy 85.09 104.14)
+		)
+		(stroke
+			(width 0)
+			(type default)
+		)
+	)
+	(wire
+		(pts
 			(xy 40.64 63.5) (xy 67.31 63.5)
 		)
@@
 	(wire
 		(pts
-			(xy 82.55 87.63) (xy 69.85 87.63)
+			(xy 85.09 87.63) (xy 81.28 87.63)
 		)
 		(stroke
@@
 		)
 		(property "Datasheet" "~"
-			(at 204.47 96.52 0)
+			(at 208.026 99.822 0)
 			(effects
 				(font
@@
 		(pin "8"
 		)
-		(pin "10"
-		)
-		(pin "11"
-		)
-		(pin "15"
-		)
-		(pin "16"
-		)
-		(pin "20"
-		)
-		(pin "4"
-		)
-		(pin "5"
-		)
-		(pin "6"
-		)
 		(instances
 			(project "PSE"
@@
 	)
 	(symbol
+		(lib_id "power:PWR_FLAG")
+		(at 81.28 87.63 0)
+		(unit 1)
+		(exclude_from_sim no)
+		(in_bom yes)
+		(on_board yes)
+		(dnp no)
+		(fields_autoplaced yes)
+		(property "Reference" "#FLG02"
+			(at 81.28 85.725 0)
+			(effects
+				(font
+					(size 1.27 1.27)
+				)
+				(hide yes)
+			)
+		)
+		(property "Value" "PWR_FLAG"
+			(at 81.28 82.55 0)
+			(effects
+				(font
+					(size 1.27 1.27)
+				)
+			)
+		)
+		(property "Footprint" ""
+			(at 81.28 87.63 0)
+			(effects
+				(font
+					(size 1.27 1.27)
+				)
+				(hide yes)
+			)
+		)
+		(property "Datasheet" "~"
+			(at 81.28 87.63 0)
+			(effects
+				(font
+					(size 1.27 1.27)
+				)
+				(hide yes)
+			)
+		)
+		(property "Description" "Special symbol for telling ERC where power comes from"
+			(at 81.28 87.63 0)
+			(effects
+				(font
+					(size 1.27 1.27)
+				)
+				(hide yes)
+			)
+		)
+		(pin "1"
+		)
+		(instances
+			(project ""
+				(path "/13844229-b559-4868-a710-53f590233cb2/bb0efcd1-04c2-4746-a524-ab8f9ddb53e9"
+					(reference "#FLG02")
+					(unit 1)
+				)
+			)
+		)
+	)
+	(symbol
 		(lib_id "Sensor_Temperature:MCP9700Ax-ETT")
 		(at 170.18 49.53 0)
@@
 	)
 	(symbol
+		(lib_name "VDD_1")
 		(lib_id "power:VDD")
 		(at 19.05 85.09 0)
@@
 			)
 		)
-		(property "Value" "VDD"
+		(property "Value" "+3V3"
 			(at 19.05 80.01 0)
 			(effects
@@
 	)
 	(symbol
-		(lib_id "Transistor_FET:Q_NMOS_SGD")
-		(at 45.72 90.17 90)
+		(lib_id "power:GND")
+		(at 153.67 146.05 0)
 		(unit 1)
 		(exclude_from_sim no)
@@
 		(dnp no)
 		(fields_autoplaced yes)
-		(property "Reference" "Q3"
-			(at 45.72 81.28 90)
+		(property "Reference" "#PWR098"
+			(at 153.67 152.4 0)
 			(effects
 				(font
 					(size 1.27 1.27)
 				)
+				(hide yes)
 			)
 		)
-		(property "Value" "IRLML9301"
-			(at 45.72 83.82 90)
+		(property "Value" "GND"
+			(at 153.67 151.13 0)
 			(effects
 				(font
@@
 			)
 		)
-		(property "Footprint" "Package_TO_SOT_SMD:SOT-23"
-			(at 43.18 85.09 0)
+		(property "Footprint" ""
+			(at 153.67 146.05 0)
 			(effects
 				(font
@@
 			)
 		)
-		(property "Datasheet" "~"
-			(at 45.72 90.17 0)
+		(property "Datasheet" ""
+			(at 153.67 146.05 0)
 			(effects
 				(font
@@
 			)
 		)
-		(property "Description" "N-MOSFET transistor, source/gate/drain"
-			(at 45.72 90.17 0)
+		(property "Description" "Power symbol creates a global label with name \"GND\" , ground"
+			(at 153.67 146.05 0)
 			(effects
 				(font
@@
 		(pin "1"
 		)
-		(pin "3"
-		)
-		(pin "2"
-		)
 		(instances
 			(project "PSE"
 				(path "/13844229-b559-4868-a710-53f590233cb2/bb0efcd1-04c2-4746-a524-ab8f9ddb53e9"
-					(reference "Q3")
+					(reference "#PWR098")
 					(unit 1)
 				)
@@
 	)
 	(symbol
-		(lib_id "power:GND")
-		(at 153.67 146.05 0)
+		(lib_id "Transistor_FET:IRLML9301")
+		(at 44.45 88.9 0)
 		(unit 1)
 		(exclude_from_sim no)
@@
 		(dnp no)
 		(fields_autoplaced yes)
-		(property "Reference" "#PWR098"
-			(at 153.67 152.4 0)
+		(property "Reference" "Q3"
+			(at 45.72 81.28 0)
 			(effects
 				(font
 					(size 1.27 1.27)
 				)
-				(hide yes)
 			)
 		)
-		(property "Value" "GND"
-			(at 153.67 151.13 0)
+		(property "Value" "IRLML9301"
+			(at 45.72 83.82 0)
 			(effects
 				(font
@@
 			)
 		)
-		(property "Footprint" ""
-			(at 153.67 146.05 0)
+		(property "Footprint" "Package_TO_SOT_SMD:SOT-23"
+			(at 62.484 76.327 0)
 			(effects
 				(font
 					(size 1.27 1.27)
+					(italic yes)
 				)
+				(justify left)
 				(hide yes)
 			)
 		)
-		(property "Datasheet" ""
-			(at 153.67 146.05 0)
+		(property "Datasheet" "https://www.infineon.com/dgdl/irlml9301pbf.pdf?fileId=5546d462533600a401535668e5e42640"
+			(at 62.484 78.232 0)
 			(effects
 				(font
 					(size 1.27 1.27)
 				)
+				(justify left)
 				(hide yes)
 			)
 		)
-		(property "Description" "Power symbol creates a global label with name \"GND\" , ground"
-			(at 153.67 146.05 0)
+		(property "Description" "-3.6A Id, -30V Vds, 64mOhm Rds, P-Channel HEXFET Power MOSFET, SOT-23"
+			(at 57.404 74.422 0)
 			(effects
 				(font
@@
 			)
 		)
+		(pin "2"
+		)
+		(pin "3"
+		)
 		(pin "1"
 		)
 		(instances
-			(project "PSE"
+			(project ""
 				(path "/13844229-b559-4868-a710-53f590233cb2/bb0efcd1-04c2-4746-a524-ab8f9ddb53e9"
-					(reference "#PWR098")
+					(reference "Q3")
 					(unit 1)
 				)

Commit message: update
Parts:
- removed J10: SERVO_3, Connector_PinHeader_2.54mm:PinHeader_1x03_P2.54mm_Vertical, symbol Connector:Conn_01x03_Pin
- removed J6: I2C_3V3, Connector_JST:JST_XH_B4B-XH-A_1x04_P2.50mm_Vertical, symbol Connector:Conn_01x04_Pin
- removed J7: UART0_3V3, Connector_JST:JST_XH_B4B-XH-A_1x04_P2.50mm_Vertical, symbol Connector:Conn_01x04_Pin
- removed J8: SERVO_1, Connector_PinHeader_2.54mm:PinHeader_1x03_P2.54mm_Vertical, symbol Connector:Conn_01x03_Pin
- removed J9: SERVO_2, Connector_PinHeader_2.54mm:PinHeader_1x03_P2.54mm_Vertical, symbol Connector:Conn_01x03_Pin
- added J10: SERVO_3, Connector_PinHeader_2.54mm:PinHeader_1x03_P2.54mm_Vertical, symbol Connector_Generic:Conn_01x03
- added J6: I2C_3V3, Connector_JST:JST_XH_B4B-XH-A_1x04_P2.50mm_Vertical, symbol Connector_Generic:Conn_01x04
- added J7: UART0_3V3, Connector_JST:JST_XH_B4B-XH-A_1x04_P2.50mm_Vertical, symbol Connector_Generic:Conn_01x04
- added J8: SERVO_1, Connector_PinHeader_2.54mm:PinHeader_1x03_P2.54mm_Vertical, symbol Connector_Generic:Conn_01x03
- added J9: SERVO_2, Connector_PinHeader_2.54mm:PinHeader_1x03_P2.54mm_Vertical, symbol Connector_Generic:Conn_01x03
- C41, C42, C43, C44, C45, C46, C48: footprint Capacitor_Tantalum_SMD:CP_EIA-1608-08_AVX-J -> Capacitor_SMD:C_0603_1608Metric
- C47: value C -> 100n; footprint Capacitor_Tantalum_SMD:CP_EIA-1608-08_AVX-J -> Capacitor_SMD:C_0603_1608Metric
- R24, R25, R26, R27, R28: footprint Resistor_SMD:R_0201_0603Metric -> Resistor_SMD:R_0603_1608Metric
- U8: footprint Package_DFN_QFN:DFN-10_2x2mm_P0.4mm -> libs:QFN16_FRE
- U9: footprint RF_Module:ESP-07 -> Connector_PinSocket_2.54mm:PinSocket_2x04_P2.54mm_Vertical
Connections:
- net +3V3: now also J6.1 (Pin_1), J7.1 (Pin_1)
- net +5V: now also J10.2 (Pin_2), J8.2 (Pin_2), J9.2 (Pin_2)
- net EXT_I2C_SCL: now also J6.2 (Pin_2)
- net EXT_I2C_SDA: now also J6.3 (Pin_3)
- net GND: now also J10.3 (Pin_3), J6.4 (Pin_4), J7.4 (Pin_4), J8.3 (Pin_3), J9.3 (Pin_3)
- net RX_SAM: now also J7.3 (Pin_3)
- net SERVO_1: now also J8.1 (Pin_1)
- net SERVO_2: now also J9.1 (Pin_1)
- net SERVO_3: now also J10.1 (Pin_1)
- net TX_SAM: now also J7.2 (Pin_2)
Other:
- moved on the sheet: C46, C48, R28, U10

Commit message: update
Parts:
- removed Q3: IRLML9301, Package_TO_SOT_SMD:SOT-23, symbol Transistor_FET:IRLML9301
- removed U7: SAM-M8Q, RF_GPS:ublox_SAM-M8Q, symbol RF_GPS:SAM-M8Q
- removed U8: MMA8451Q, libs:QFN16_FRE, symbol Sensor_Motion:MMA8653FCR1
- removed U9: ESP-01, Connector_PinSocket_2.54mm:PinSocket_2x04_P2.54mm_Vertical, symbol RF_Module:ESP-07
- added Q1: IRLML9301, Package_TO_SOT_SMD:SOT-23, symbol libs:IRLML9301
- added U7: SAM-M8Q, RF_GPS:ublox_SAM-M8Q, symbol libs:SAM-M8Q
- added U8: MMA8451Q, libs:QFN16_FRE, symbol libs:MMA8653FCR1
- added U9: ESP-01, Connector_PinSocket_2.54mm:PinSocket_2x04_P2.54mm_Vertical, symbol libs:ESP-07
Connections:
- net +3V3: now also Q1.2 (S), U8.1 (VDDIO), U8.14 (VDD), U9.5 (VCC)
- net ACC_INT1: now also U8.11 (INT1)
- net ACC_INT2: now also U8.9 (INT2)
- net ACC_SCL: now also U8.4 (SCL)
- net ACC_SDA: now also U8.6 (SDA)
- net ESP_EN: now also U9.7 (EN)
- net ESP_RX: now also U9.4 (UART_RX)
- net ESP_TX: now also U9.8 (UART_TX)
- net GND: now also U7.1 (GND), U8.10 (GND), U8.12 (GND), U8.5 (GND), U8.7 (SAO), U9.1 (GND)
- net RX_SAM: now also U7.14 (RXD)
- net SAM_EN: now also Q1.1 (G)
- net SAM_PPS: now also U7.7 (TIMEPULSE)
- net SAM_RST: now also U7.18 (~{RESET})
- net TX_SAM: now also U7.13 (TXD)
- net at C42.1, C44.1: now also Q1.3 (D), U7.17 (VCC), U7.2 (VCC_IO), U7.3 (V_BCKP)
- net at C43.1: now also U8.2 (BYP)
- net at R27.2: now also U9.6 (~{RST})

Commit message: update
Other:
- title: (none) -> Sensoristica ed Espansioni
Changed lines of the file:
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@@
 	(generator_version "9.0")
 	(paper "A4")
+	(title_block
+		(title "Sensoristica ed Espansioni")
+	)
 	(rectangle
 		(start 15.24 144.78)

Commit message: update
Parts:
- renumbered Q1 to Q3
Changed lines of the file:
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@@
 		(dnp no)
 		(fields_autoplaced yes)
-		(property "Reference" "Q1"
+		(property "Reference" "Q3"
 			(at 45.72 81.28 0)
 			(effects
@@
 			(project ""
 				(path "/13844229-b559-4868-a710-53f590233cb2/bb0efcd1-04c2-4746-a524-ab8f9ddb53e9"
-					(reference "Q1")
+					(reference "Q3")
 					(unit 1)
 				)
