File: hard/PSE.kicad_pcb (KiCad board)
At the start: 2 copper layers, 0 parts

Commit message: update
Parts:
- added BZ1: Buzzer, Buzzer_Beeper:Buzzer_12x9.5RM7.6, F.Cu at (185.0, 97.5)
- added C1: 100n, Capacitor_Tantalum_SMD:CP_EIA-1608-08_AVX-J, F.Cu at (175.2, 71.0)
- added C10: 100n, Capacitor_Tantalum_SMD:CP_EIA-1608-08_AVX-J, F.Cu at (143.0, 96.0)
- added C11: 100n, Capacitor_Tantalum_SMD:CP_EIA-1608-08_AVX-J, F.Cu at (166.0, 77.9)
- added C12: 100n, Capacitor_Tantalum_SMD:CP_EIA-1608-08_AVX-J, F.Cu at (142.0, 82.0)
- added C13: 100n, Capacitor_Tantalum_SMD:CP_EIA-1608-08_AVX-J, F.Cu at (143.5, 80.5)
- added C14: 100n, Capacitor_Tantalum_SMD:CP_EIA-1608-08_AVX-J, F.Cu at (162.0, 85.0)
- added C15: 100n, Capacitor_Tantalum_SMD:CP_EIA-1608-08_AVX-J, F.Cu at (141.5, 93.5)
- added C16: 100n, Capacitor_Tantalum_SMD:CP_EIA-1608-08_AVX-J, F.Cu at (140.5, 83.5)
- added C17: 100n, Capacitor_Tantalum_SMD:CP_EIA-1608-08_AVX-J, F.Cu at (154.5, 82.5)
- added C18: 100n, Capacitor_Tantalum_SMD:CP_EIA-1608-08_AVX-J, F.Cu at (151.5, 80.0)
- added C19: 2.2u, Capacitor_Tantalum_SMD:CP_EIA-1608-08_AVX-J, F.Cu at (150.0, 78.5)
- added C2: 100n, Capacitor_Tantalum_SMD:CP_EIA-1608-08_AVX-J, F.Cu at (191.0, 80.3)
- added C20: 2.2u, Capacitor_Tantalum_SMD:CP_EIA-1608-08_AVX-J, F.Cu at (148.5, 77.0)
- added C21: DNP 100n, Capacitor_Tantalum_SMD:CP_EIA-1608-08_AVX-J, F.Cu at (127.5, 78.0)
- added C22: 18p, Capacitor_Tantalum_SMD:CP_EIA-1608-08_AVX-J, F.Cu at (158.0, 97.0)
- added C23: 18p, Capacitor_Tantalum_SMD:CP_EIA-1608-08_AVX-J, F.Cu at (160.0, 91.0)
- added C24: 100n, Capacitor_Tantalum_SMD:CP_EIA-1608-08_AVX-J, F.Cu at (176.0, 82.2)
- added C25: 100n, Capacitor_Tantalum_SMD:CP_EIA-1608-08_AVX-J, F.Cu at (164.5, 101.8)
- added C26: 100n, Capacitor_Tantalum_SMD:CP_EIA-1608-08_AVX-J, F.Cu at (199.5, 110.3)
- added C27: 100n, Capacitor_Tantalum_SMD:CP_EIA-1608-08_AVX-J, F.Cu at (170.5, 111.7)
- added C28: 4.7u, Capacitor_Tantalum_SMD:CP_EIA-1608-08_AVX-J, F.Cu at (142.0, 104.0)
- added C29: 100n, Capacitor_Tantalum_SMD:CP_EIA-1608-08_AVX-J, F.Cu at (140.0, 104.1)
- added C3: 100n, Capacitor_Tantalum_SMD:CP_EIA-1608-08_AVX-J, F.Cu at (189.5, 118.8)
- added C30: 10u, Capacitor_Tantalum_SMD:CP_EIA-1608-08_AVX-J, F.Cu at (103.1, 98.6)
- added C31: 10u, Capacitor_Tantalum_SMD:CP_EIA-1608-08_AVX-J, F.Cu at (105.0, 98.6)
- added C32: 100n, Capacitor_Tantalum_SMD:CP_EIA-1608-08_AVX-J, F.Cu at (107.0, 98.6)
- added C33: 1u, Capacitor_Tantalum_SMD:CP_EIA-1608-08_AVX-J, F.Cu at (114.6, 93.1)
- added C34: 1u, Capacitor_Tantalum_SMD:CP_EIA-1608-08_AVX-J, F.Cu at (107.1, 93.1)
- added C35: 100n, Capacitor_Tantalum_SMD:CP_EIA-1608-08_AVX-J, F.Cu at (120.3, 111.5)
- added C36: 2.2u, Capacitor_Tantalum_SMD:CP_EIA-1608-08_AVX-J, F.Cu at (163.6, 72.6)
- added C37: 22u, Capacitor_Tantalum_SMD:CP_EIA-1608-08_AVX-J, F.Cu at (117.2, 100.0)
- added C38: 100n, Capacitor_Tantalum_SMD:CP_EIA-1608-08_AVX-J, F.Cu at (129.5, 119.8)
- added C39: 22u, Capacitor_Tantalum_SMD:CP_EIA-1608-08_AVX-J, F.Cu at (117.2, 97.5)
- added C4: 100n, Capacitor_Tantalum_SMD:CP_EIA-1608-08_AVX-J, F.Cu at (180.5, 127.5)
- added C40: 100n, Capacitor_Tantalum_SMD:CP_EIA-1608-08_AVX-J, F.Cu at (117.2, 95.0)
- added C41: 100n, Capacitor_Tantalum_SMD:CP_EIA-1608-08_AVX-J, F.Cu at (134.3, 110.7)
- added C42: 4u7, Capacitor_Tantalum_SMD:CP_EIA-1608-08_AVX-J, F.Cu at (151.1, 103.7)
- added C43: 100n, Capacitor_Tantalum_SMD:CP_EIA-1608-08_AVX-J, F.Cu at (136.0, 110.7)
- added C44: 100n, Capacitor_Tantalum_SMD:CP_EIA-1608-08_AVX-J, F.Cu at (149.1, 103.7)
- added C45: 4.7u, Capacitor_Tantalum_SMD:CP_EIA-1608-08_AVX-J, F.Cu at (132.0, 106.5)
- added C46: 100n, Capacitor_Tantalum_SMD:CP_EIA-1608-08_AVX-J, F.Cu at (160.5, 66.9)
- added C47: C, Capacitor_Tantalum_SMD:CP_EIA-1608-08_AVX-J, F.Cu at (114.0, 79.8)
- added C48: 1u 6V3, Capacitor_Tantalum_SMD:CP_EIA-1608-08_AVX-J, F.Cu at (161.2, 69.5)
- added C5: 100n, Capacitor_Tantalum_SMD:CP_EIA-1608-08_AVX-J, F.Cu at (126.3, 127.5)
- added C6: 100n, Capacitor_Tantalum_SMD:CP_EIA-1608-08_AVX-J, F.Cu at (109.0, 116.2)
- added C7: 100n, Capacitor_Tantalum_SMD:CP_EIA-1608-08_AVX-J, F.Cu at (110.1, 87.6)
- added C8: 100n, Capacitor_Tantalum_SMD:CP_EIA-1608-08_AVX-J, F.Cu at (125.5, 71.0)
- added C9: 100n, Capacitor_Tantalum_SMD:CP_EIA-1608-10_AVX-L, F.Cu at (160.5, 86.5)
- added D1: WS2812B, LED_SMD:LED_WS2812B_PLCC4_5.0x5.0mm_P3.2mm, F.Cu at (175.5, 66.0)
- added D10: LED_alive, LED_SMD:LED_0805_2012Metric, F.Cu at (158.6, 81.5)
- added D11: TVS VBR 17V IBR=1mA, Diode_SMD:D_SMA, F.Cu at (112.0, 118.0)
- added D12: S1B, Diode_SMD:D_SMA, F.Cu at (111.0, 109.0)
- added D13: RBR1VWM30ATFTR, Diode_SMD:D_SOD-123, F.Cu at (134.0, 65.7)
- added D14: 1N4148, Diode_SMD:D_SOD-123, F.Cu at (140.8, 113.5)
- added D15: 1N4148, Diode_SMD:D_SOD-123F, F.Cu at (137.1, 119.0)
- added D16: 3V3_LED, LED_SMD:LED_0805_2012Metric, F.Cu at (115.0, 87.4)
- added D17: PDZ3.3B.115, Diode_SMD:D_SOD-323_HandSoldering, F.Cu at (131.5, 119.8)
- added D18: 5V_LED, LED_SMD:LED_0805_2012Metric_Pad1.15x1.40mm_HandSolder, F.Cu at (117.0, 87.5)
- added D19: RBR1VWM30ATFTR, Diode_SMD:D_SOD-123, F.Cu at (146.5, 125.0)
- added D2: WS2812B, LED_SMD:LED_WS2812B_PLCC4_5.0x5.0mm_P3.2mm, F.Cu at (196.0, 82.0)
- added D3: WS2812B, LED_SMD:LED_WS2812B_PLCC4_5.0x5.0mm_P3.2mm, F.Cu at (196.5, 117.0)
- added D4: WS2812B, LED_SMD:LED_WS2812B_PLCC4_5.0x5.0mm_P3.2mm, F.Cu at (178.5, 132.5)
- added D5: WS2812B, LED_SMD:LED_WS2812B_PLCC4_5.0x5.0mm_P3.2mm, F.Cu at (124.5, 132.0)
- added D6: WS2812B, LED_SMD:LED_WS2812B_PLCC4_5.0x5.0mm_P3.2mm, F.Cu at (105.0, 115.5)
- added D7: WS2812B, LED_SMD:LED_WS2812B_PLCC4_5.0x5.0mm_P3.2mm, F.Cu at (105.5, 82.5)
- added D8: WS2812B, LED_SMD:LED_WS2812B_PLCC4_5.0x5.0mm_P3.2mm, F.Cu at (127.1, 65.5)
- added D9: 1N4148, Diode_SMD:D_SOD-123, F.Cu at (189.5, 90.9)
- added F1: 2016L05MR, Fuse:Fuse_1206_3216Metric, F.Cu at (106.1, 108.0)
- added FB1: FerriteBead, Capacitor_SMD:C_0805_2012Metric, F.Cu at (133.1, 71.5)
- added J10: SERVO_3, Connector_PinHeader_2.54mm:PinHeader_1x03_P2.54mm_Vertical, F.Cu at (183.5, 117.0)
- added J2: Conn_01x03, Connector_PinHeader_2.54mm:PinHeader_1x03_P2.54mm_Vertical, F.Cu at (169.5, 93.5)
- added J4: USB_B_Mini, Connector_USB:USB_Mini-B_Wuerth_65100516121_Horizontal, F.Cu at (151.3, 67.4)
- added J6: I2C_3V3, Connector_JST:JST_XH_B4B-XH-A_1x04_P2.50mm_Vertical, F.Cu at (161.8, 130.5)
- added J7: UART0_3V3, Connector_JST:JST_XH_B4B-XH-A_1x04_P2.50mm_Vertical, F.Cu at (136.5, 130.5)
- added J8: SERVO_1, Connector_PinHeader_2.54mm:PinHeader_1x03_P2.54mm_Vertical, F.Cu at (176.0, 116.9)
- added J9: SERVO_2, Connector_PinHeader_2.54mm:PinHeader_1x03_P2.54mm_Vertical, F.Cu at (179.9, 117.0)
- added L1: 2.2u, Capacitor_SMD:C_0603_1608Metric, F.Cu at (117.2, 102.5)
- added Q2: PDTC114YT, Package_TO_SOT_SMD:SOT-23, F.Cu at (189.4, 86.2)
- added Q3: IRLML9301, Package_TO_SOT_SMD:SOT-23, F.Cu at (155.1, 103.5)
- added Q4: IRLML9301, Package_TO_SOT_SMD:SOT-23, F.Cu at (138.6, 67.0)
- added R1: 1k, Resistor_SMD:R_0603_1608Metric, F.Cu at (167.0, 65.0)
- added R10: R, Resistor_SMD:R_0603_1608Metric, F.Cu at (149.5, 99.0)
- added R11: 470k, Resistor_SMD:R_0603_1608Metric, F.Cu at (151.0, 99.0)
- added R12: 470, Resistor_SMD:R_0603_1608Metric, F.Cu at (156.0, 84.0)
- added R13: 27, Resistor_SMD:R_0603_1608Metric, F.Cu at (143.0, 71.3)
- added R14: 27, Resistor_SMD:R_0603_1608Metric, F.Cu at (142.9, 74.5)
- added R15: 10k, Resistor_SMD:R_0603_1608Metric, F.Cu at (116.3, 117.0)
- added R16: 510, Resistor_SMD:R_0603_1608Metric, F.Cu at (112.0, 87.7)
- added R17: 10k, Resistor_SMD:R_0603_1608Metric, F.Cu at (119.0, 114.3)
- added R18: 1.8k, Resistor_SMD:R_0603_1608Metric, F.Cu at (103.8, 101.3)
- added R19: 200, Resistor_SMD:R_0603_1608Metric, F.Cu at (159.5, 71.5)
- added R20: 150k, Resistor_SMD:R_0603_1608Metric, F.Cu at (127.2, 121.0)
- added R21: 56k, Resistor_SMD:R_0603_1608Metric, F.Cu at (128.7, 122.5)
- added R22: 1k, Resistor_SMD:R_0603_1608Metric, F.Cu at (127.2, 119.5)
- added R23: 510, Resistor_SMD:R_0603_1608Metric, F.Cu at (119.5, 87.7)
- added R24: 10k, Resistor_SMD:R_0603_1608Metric, F.Cu at (159.0, 103.6)
- added R25: 4.7k, Resistor_SMD:R_0603_1608Metric, F.Cu at (133.0, 95.2)
- added R26: 4.7k, Resistor_SMD:R_0603_1608Metric, F.Cu at (131.5, 95.2)
- added R27: 10k, Resistor_SMD:R_0603_1608Metric, F.Cu at (114.1, 74.5)
- added R28: 470, Resistor_SMD:R_0603_1608Metric, F.Cu at (162.4, 66.7)
- added R29: 10k, Resistor_SMD:R_0603_1608Metric, F.Cu at (143.1, 67.2)
- added R30: 47k, Resistor_SMD:R_0603_1608Metric, F.Cu at (138.2, 75.0)
- added R4: 10k, Resistor_SMD:R_0603_1608Metric, F.Cu at (165.8, 75.5)
- added R5: 10k, Resistor_SMD:R_0603_1608Metric, F.Cu at (125.0, 93.7)
- added R6: 1k, Resistor_SMD:R_0603_1608Metric, F.Cu at (123.0, 93.7)
- added R7: R, Resistor_SMD:R_0603_1608Metric, F.Cu at (155.4, 90.6)
- added R8: 470k, Resistor_SMD:R_0603_1608Metric, F.Cu at (146.5, 99.0)
- added R9: 470k, Resistor_SMD:R_0603_1608Metric, F.Cu at (148.0, 99.0)
- added REF**: MountingHole_3.2mm_M3_Pad_Via, MountingHole:MountingHole_3.2mm_M3_Pad_Via, F.Cu at (112.6, 133.9)
- added REF**: MountingHole_3.2mm_M3_Pad_Via, MountingHole:MountingHole_3.2mm_M3_Pad_Via, F.Cu at (112.6, 65.9)
- added REF**: MountingHole_3.2mm_M3_Pad_Via, MountingHole:MountingHole_3.2mm_M3_Pad_Via, F.Cu at (189.5, 65.9)
- added REF**: MountingHole_3.2mm_M3_Pad_Via, MountingHole:MountingHole_3.2mm_M3_Pad_Via, F.Cu at (189.6, 133.9)
- added SW1: RESET_SW, Button_Switch_SMD:SW_SPST_EVQP0, F.Cu at (172.1, 76.4)
- added SW2: PROG_SW, Button_Switch_SMD:SW_SPST_EVQP0, F.Cu at (184.0, 76.4)
- added SW3: SW_U, Button_Switch_SMD:SW_SPST_EVQP0, F.Cu at (181.0, 85.9)
- added SW4: SW_L, Button_Switch_SMD:SW_SPST_EVQP0, F.Cu at (170.0, 99.8)
- added SW5: SW_R, Button_Switch_SMD:SW_SPST_EVQP0, F.Cu at (192.1, 99.8)
- added SW6: SW_D, Button_Switch_SMD:SW_SPST_EVQP0, F.Cu at (181.5, 108.4)
- added SW7: Power_button, Button_Switch_SMD:SW_SPST_EVQP0, F.Cu at (143.0, 118.0)
- added TP4: 3V3A, TestPoint:TestPoint_THTPad_D1.5mm_Drill0.7mm, F.Cu at (160.5, 74.0)
- added U1: RP2040, Package_DFN_QFN:QFN-56-1EP_7x7mm_P0.4mm_EP3.2x3.2mm, F.Cu at (148.0, 90.0)
- added U10: TC1047A, Package_TO_SOT_SMD:SOT-23, F.Cu at (161.5, 62.9)
- added U2: W25Q128JVE, Package_SON:WSON-8-1EP_8x6mm_P1.27mm_EP3.4x4.3mm, F.Cu at (130.6, 85.8)
- added U3: AT24C256, Package_SO:SOIC-8_3.9x4.9mm_P1.27mm, F.Cu at (127.4, 110.0)
- added U4: oled_0.96"_128x64px, Connector_PinHeader_2.54mm:PinHeader_1x04_P2.54mm_Vertical, F.Cu at (133.0, 99.5)
- added U5: XC6705A331MR-G, Package_TO_SOT_SMD:SOT-23-5, F.Cu at (110.6, 93.1)
- added U6: TPS563201, Package_SO:SOIC-8_3.9x4.9mm_P1.27mm, F.Cu at (111.5, 100.9)
- added U7: SAM-M8Q, RF_GPS:ublox_SAM-M8Q, F.Cu at (159.5, 116.0)
- added U8: MMA8451Q, Package_DFN_QFN:DFN-10_2x2mm_P0.4mm, F.Cu at (136.7, 106.5)
- added U9: ESP-01, Connector_PinSocket_2.54mm:PinSocket_2x04_P2.54mm_Vertical, F.Cu at (121.0, 72.9)
- added Y1: 12MHz, Crystal:Crystal_SMD_3225-4Pin_3.2x2.5mm_HandSoldering, F.Cu at (155.7, 94.7)
Routing:
- net +3V3: track 0.00 -> 223.6 mm
- net VDD: track 0.00 -> 40.9 mm
- net +12V: track 0.00 -> 14.1 mm
- net +1V1: track 0.00 -> 12.3 mm
- net Net-(U9-~{RST}): track 0.00 -> 6.18 mm
- net +3V3A: track 0.00 -> 6.02 mm
- added copper zone on B.Cu, net GND
- added copper zone on F.Cu, net GND
Other:
- board outline added: 102.2 x 77.2 mm
- board text added: "${REFERENCE}"
