File: hard/PSE.kicad_pcb (KiCad board)
At the start: 2 copper layers, 102.2 x 77.2 mm, 132 parts, among them J10 SERVO_3, J2 Conn_01x03, J4 USB_B_Mini, J6 I2C_3V3, J7 UART0_3V3, J8 SERVO_1, J9 SERVO_2, Q2 PDTC114YT, Q3 IRLML9301, Q4 IRLML9301, SW1 RESET_SW, SW2 PROG_SW, SW3 SW_U, SW4 SW_L, SW5 SW_R, SW6 SW_D, SW7 Power_button, U1 RP2040, U10 TC1047A, U2 W25Q128JVE, U3 AT24C256, U4 oled_0.96"_128x64px, U5 XC6705A331MR-G, U6 TPS563201, U7 SAM-M8Q, U8 MMA8451Q, U9 ESP-01, Y1 12MHz

Commit message: update
Connections:
- J2 pad 2: (no net) -> GND
- J2 pad 3: (no net) -> /mcu/SWCLK
Routing:
- net +5V: track 0.00 -> 320.0 mm, vias 0 -> 2
- net +12V: track 14.1 -> 55.4 mm, vias 0 -> 2
- net GND: vias 0 -> 1

Commit message: update
Parts:
- moved J6 3.77 mm to (159.5, 133.5)
- moved J7 2.92 mm to (135.0, 133.0)
Other:
- board text added: "GND SDA SCL 3V3"
- board text added: "I2C"
Changed lines of the file:
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@@
 	(footprint "Connector_JST:JST_XH_B4B-XH-A_1x04_P2.50mm_Vertical"
 		(layer "F.Cu")
-		(at 136.5 130.5)
+		(at 135 133)
 		(descr "JST XH series connector, B4B-XH-A (http://www.jst-mfg.com/product/pdf/eng/eXH.pdf), generated with kicad-footprint-generator")
 		(tags "connector JST XH vertical")
@@
 		(tags "SOD-123")
 		(property "Reference" "D13"
-			(at -3.65 0 180)
+			(at -3.65 0 0)
 			(layer "F.SilkS")
 			(effects
@@
 	(footprint "Connector_JST:JST_XH_B4B-XH-A_1x04_P2.50mm_Vertical"
 		(layer "F.Cu")
-		(at 161.75 130.475)
+		(at 159.5 133.5)
 		(descr "JST XH series connector, B4B-XH-A (http://www.jst-mfg.com/product/pdf/eng/eXH.pdf), generated with kicad-footprint-generator")
 		(tags "connector JST XH vertical")
 		(property "Reference" "J6"
-			(at 3.75 -3.55 0)
+			(at 11 0.5 0)
 			(layer "F.SilkS")
 			(effects
@@
 		(layer "Edge.Cuts")
 	)
+	(gr_text "I2C"
+		(at 166.5 128 0)
+		(layer "F.SilkS" knockout)
+		(effects
+			(font
+				(size 1.5 1.5)
+				(thickness 0.3)
+				(bold yes)
+			)
+			(justify left bottom)
+		)
+	)
+	(gr_text "GND SDA SCL 3V3"
+		(at 164 130 0)
+		(layer "F.SilkS" knockout)
+		(effects
+			(font
+				(size 1 1)
+				(thickness 0.25)
+				(bold yes)
+			)
+			(justify bottom)
+		)
+	)
 	(gr_text "${REFERENCE}"

Commit message: update
Parts:
- moved C48 7.32 mm to (168.5, 70.0), turned to -90 degrees
- moved C15 7.20 mm to (137.5, 99.5)
- moved C10 6.40 mm to (139.0, 101.0)
- moved C16 6.00 mm to (136.5, 79.0)
- moved C12 5.78 mm to (138.0, 77.8)
- moved C22 5.57 mm to (163.1, 99.3)
- moved Y1 5.52 mm to (160.5, 97.4)
- moved C8 5.32 mm to (121.5, 67.5)
- moved C33 4.37 mm to (118.4, 91.0)
- moved SW5 4.35 mm to (196.3, 98.8)
- moved C44 4.33 mm to (150.2, 107.9)
- moved U4 4.14 mm to (128.9, 99.8)
- moved C23 3.71 mm to (163.1, 89.0)
- moved R26 3.52 mm to (128.0, 95.2)
- moved R24 3.30 mm to (162.3, 103.8)
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Routing:
- net Net-(D4-DOUT): track 0.00 -> 59.9 mm
- net /I2C0_SCL: track 0.00 -> 58.8 mm, vias 0 -> 4
- net /ui/BUTTON_U: track 0.00 -> 58.2 mm, vias 0 -> 4
- net Net-(U1-RUN): track 0.00 -> 56.1 mm, vias 0 -> 4
- net /I2C0_SDA: track 0.00 -> 46.6 mm, vias 0 -> 2
- net /mcu/UART0_TX: track 0.00 -> 46.6 mm, vias 0 -> 2
- net /mcu/BUZZER_PWM: track 0.00 -> 45.1 mm
- net /power/BUCK_EN: track 0.00 -> 43.9 mm, vias 0 -> 4
- net /mcu/VBAT: track 0.00 -> 42.4 mm, vias 0 -> 2
- net /mcu/UART0_RX: track 0.00 -> 41.2 mm, vias 0 -> 2
- net /mcu/PWM_SERVO3: track 0.00 -> 41.1 mm, vias 0 -> 1
- net Net-(D2-DOUT): track 0.00 -> 40.3 mm, vias 0 -> 2
- net Net-(D6-DOUT): track 0.00 -> 40.0 mm, vias 0 -> 2
- net Net-(Q3-S): track 0.00 -> 39.9 mm
- net /ui/BUTTON_L: track 0.00 -> 39.8 mm, vias 0 -> 1
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Other:
- board text removed: "${REFERENCE}"

Commit message: update
Parts:
- removed TP4: 3V3A, TestPoint:TestPoint_THTPad_D1.5mm_Drill0.7mm
- J2: moved to B.Cu
- moved C14 10.8 mm to (155.2, 93.4)
- moved C9 8.06 mm to (153.7, 82.1)
- moved C23 6.37 mm to (158.3, 93.2)
- moved J2 5.53 mm to (170.6, 88.1)
- moved R7 5.29 mm to (156.6, 95.7)
- moved C20 4.32 mm to (145.7, 77.2)
- moved U1 4.31 mm to (143.7, 90.0), turned to 45 degrees
- moved C13 3.34 mm to (146.8, 79.8)
- moved C12 2.92 mm to (135.3, 79.0)
- moved U7 2.81 mm to (159.7, 118.8)
- moved C16 2.73 mm to (133.9, 80.0)
- moved U2 2.26 mm to (128.7, 84.3)
- moved C17 1.69 mm to (155.7, 79.8)
- moved R8 1.49 mm to (147.1, 101.5)
- moved R11 1.38 mm to (153.4, 101.6)
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Routing:
- net /led/DIN: track 4.44 -> 130.2 mm, vias 1 -> 2
- net Net-(R6-Pad2): track 19.7 -> 131.3 mm, vias 5 -> 4
- net /ui/BUTTON_D: track 23.1 -> 128.5 mm, vias 0 -> 4
- net /mcu/UART0_TX: track 46.6 -> 151.1 mm, vias 2 -> 1
- net /ui/BUTTON_R: track 34.9 -> 139.2 mm, vias 4 -> 6
- net +3V3: track 213.1 -> 306.6 mm, vias 12 -> 3
- net /mcu/UART0_RX: track 41.2 -> 109.1 mm, vias 2 -> 1
- net Net-(U1-RUN): track 56.1 -> 119.9 mm, vias 4 -> 2
- net /mcu/PWM_SERVO2: track 2.28 -> 57.3 mm, vias 0 -> 2
- net /mcu/PWM_SERVO1: track 2.08 -> 56.0 mm, vias 0 -> 2
- net /mcu/5V_EN: track 2.49 -> 53.3 mm, vias 0 -> 2
- net /mcu/USB_ID: track 5.92 -> 50.9 mm, vias 0 -> 2
- net +5V: track 292.9 -> 336.8 mm, vias 15 -> 6
- net /mcu/SWDIO: track 2.61 -> 39.1 mm, vias 0 -> 1
- net +1V1: track 21.5 -> 57.6 mm, vias 0 -> 7
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
Commit message: update
Parts:
- removed REF** (x4): MountingHole_3.2mm_M3_Pad_Via, MountingHole:MountingHole_3.2mm_M3_Pad_Via
- added H1: MountingHole, MountingHole:MountingHole_3.2mm_M3_Pad_Via, F.Cu at (112.5, 65.9)
- added H2: MountingHole, MountingHole:MountingHole_3.2mm_M3_Pad_Via, F.Cu at (189.4, 65.9)
- added H3: MountingHole, MountingHole:MountingHole_3.2mm_M3_Pad_Via, F.Cu at (112.5, 133.8)
- added H4: MountingHole, MountingHole:MountingHole_3.2mm_M3_Pad_Via, F.Cu at (189.5, 133.9)
- added J1: WS2812B, Connector_PinHeader_2.54mm:PinHeader_1x03_P2.54mm_Vertical, F.Cu at (194.7, 82.6)
- added J3: Vin, libs:TerminalBlock_bornier-2_P5.08mm, F.Cu at (106.1, 101.6)
- added J5: Vout 5V, libs:TerminalBlock_bornier-2_P5.08mm, F.Cu at (106.1, 109.7)
- added NT1: gnda-gnd, NetTie:NetTie-2_SMD_Pad0.5mm, F.Cu at (145.8, 67.0)
- added TP1: VBUS, TestPoint:TestPoint_THTPad_D1.5mm_Drill0.7mm, F.Cu at (168.4, 63.8)
- added TP2: 5V, TestPoint:TestPoint_THTPad_D1.5mm_Drill0.7mm, F.Cu at (116.0, 105.5)
- added TP3: 3V3, TestPoint:TestPoint_THTPad_D1.5mm_Drill0.7mm, F.Cu at (150.0, 64.2)
- added TP4: 3V3A, TestPoint:TestPoint_THTPad_D1.5mm_Drill0.7mm, F.Cu at (156.5, 85.8)
- C1, C10, C11, C12, C13, C14, C15, C16, C17, C18, C19, C2, C20, C21, C22, C23, C24, C25, C26, C27, C28, C29, C3, C32, C33, C34, C35, C36, C38, C4, C40, C41, C42, C43, C44, C45, C46, C48, C5, C6, C7, C8: footprint Capacitor_Tantalum_SMD:CP_EIA-1608-08_AVX-J -> Capacitor_SMD:C_0603_1608Metric
- C30, C31, C37, C39: footprint Capacitor_Tantalum_SMD:CP_EIA-1608-08_AVX-J -> Capacitor_SMD:C_0805_2012Metric
- C47: value C -> 100n; footprint Capacitor_Tantalum_SMD:CP_EIA-1608-08_AVX-J -> Capacitor_SMD:C_0603_1608Metric
- C9: footprint Capacitor_Tantalum_SMD:CP_EIA-1608-10_AVX-L -> Capacitor_SMD:C_0603_1608Metric
- D10: footprint LED_SMD:LED_0805_2012Metric -> LED_SMD:LED_0603_1608Metric
- D15: footprint Diode_SMD:D_SOD-123F -> Diode_SMD:D_SOD-123
- D18: footprint LED_SMD:LED_0805_2012Metric_Pad1.15x1.40mm_HandSolder -> LED_SMD:LED_0805_2012Metric
- J2: moved to F.Cu
- R10: value R -> 470k
- R7: value R -> 1k
- U8: footprint Package_DFN_QFN:DFN-10_2x2mm_P0.4mm -> libs:QFN16_FRE
- moved D6 94.6 mm to (198.0, 98.4), turned to 0 degrees
- moved D7 88.1 mm to (190.9, 104.0)
- moved C2 81.8 mm to (117.8, 116.8), turned to 180 degrees
- moved D8 80.7 mm to (198.0, 104.0)
- moved D5 75.8 mm to (190.9, 98.5)
- moved C3 74.7 mm to (114.8, 118.3), turned to 180 degrees
- moved C1 74.4 mm to (117.8, 118.3)
- moved R27 71.7 mm to (166.3, 123.5)
- moved U9 68.0 mm to (161.2, 127.7), turned to 180 degrees
- moved C4 66.6 mm to (114.8, 116.8), turned to 0 degrees
- moved J10 65.6 mm to (122.5, 92.8), turned to -90 degrees
- moved J9 59.9 mm to (122.5, 100.0), turned to -90 degrees
- moved J8 57.3 mm to (122.5, 96.4), turned to -90 degrees
- moved SW2 56.4 mm to (127.7, 79.3), turned to 90 degrees
- moved C38 51.2 mm to (171.1, 89.9), turned to 180 degrees
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Connections:
- net Net-(D1-DIN) renamed /led/DIN_INT
- BZ1 pad 1: VDD -> +3V3
- C36 pad 1: +3V3A -> +3.3VA
- C42 pad 1: Net-(Q3-S) -> Net-(Q3-D)
- C44 pad 1: Net-(Q3-S) -> Net-(Q3-D)
- D9 pad 1: VDD -> +3V3
- J6 pad 1: GND -> +3V3
- J6 pad 2: /I2C0_SDA -> /I2C0_SCL
- J6 pad 3: /I2C0_SCL -> /I2C0_SDA
- J6 pad 4: +3V3 -> GND
- J7 pad 1: GND -> +3V3
- J7 pad 2: /sensors/UART_TX -> /sensors/UART_RX
- J7 pad 3: /sensors/UART_RX -> /sensors/UART_TX
- J7 pad 4: +3V3 -> GND
- Q3 pad 1: Net-(Q3-S) -> /mcu/GPS_EN
- Q3 pad 2: /mcu/GPS_EN -> +3V3
- Q3 pad 3: VDD -> Net-(Q3-D)
- R19 pad 2: +3V3A -> +3.3VA
- R24 pad 1: VDD -> +3V3
- R5 pad 2: Net-(U2-~{CS}) -> /mcu/~{FLASH_CS}
- R6 pad 1: Net-(U2-~{CS}) -> /mcu/~{FLASH_CS}
- U1 pad 2: /mcu/I2CO_SDA -> /I2C0_SDA
- U1 pad 3: /mcu/I2CO_SCL -> /I2C0_SCL
- U1 pad 54: /mcu/FLASH_D2 -> /mcu/~{FLASH_D2}
- U1 pad 56: /mcu/FLASH_CS -> /mcu/~{FLASH_CS}
- U1 pad 7: /sensors/UART_LX -> /sensors/UART_RX
- U2 pad 1: Net-(U2-~{CS}) -> /mcu/~{FLASH_CS}
- U3 pad 5: /mcu/I2CO_SDA -> /I2C0_SDA
- U3 pad 6: /mcu/12CO_SCL -> /I2C0_SCL
- U4 pad 3: /mcu/I2CO_SCL -> /I2C0_SCL
- U4 pad 4: /mcu/I2CO_SDA -> /I2C0_SDA
- U7 pad 10: GND -> (no net)
- U7 pad 11: GND -> (no net)
- U7 pad 13: /sensors/UART_LX -> /sensors/UART_RX
- U7 pad 15: GND -> (no net)
- U7 pad 16: GND -> (no net)
- U7 pad 17: Net-(Q3-S) -> Net-(Q3-D)
- U7 pad 2: Net-(Q3-S) -> Net-(Q3-D)
- U7 pad 20: GND -> (no net)
- U7 pad 3: Net-(Q3-S) -> Net-(Q3-D)
- U7 pad 4: GND -> (no net)
- U7 pad 5: GND -> (no net)
- U7 pad 6: GND -> (no net)
Routing:
- net /mcu/UART0_TX: track 151.1 -> 26.1 mm, vias 1 -> 0
- net /power/VBUS: track 23.0 -> 138.6 mm
- net Net-(R6-Pad2): track 131.3 -> 16.2 mm, vias 4 -> 0
- net Net-(R20-Pad2): track 4.39 -> 114.7 mm
- net /mcu/UART0_RX: track 109.1 -> 20.3 mm, vias 1 -> 0
- net /sensors/UART_RX: track 0.00 -> 79.9 mm, vias 0 -> 1
- net /led/DIN: track 130.2 -> 52.9 mm
- net /ui/BUTTON_R: track 139.2 -> 62.8 mm, vias 6 -> 2
- net /ui/BUTTON_D: track 128.5 -> 53.0 mm, vias 4 -> 0
- net +5V: track 336.8 -> 263.0 mm, vias 6 -> 2
- net /mcu/LED_ALIVE: track 14.1 -> 87.8 mm, vias 0 -> 2
- net Net-(U1-RUN): track 119.9 -> 51.5 mm
- net Net-(Q3-D): track 0.00 -> 60.3 mm
- net Net-(D4-DOUT): track 59.9 -> 3.25 mm
- net /power/VIN: track 62.7 -> 7.27 mm
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Other:
- board text added: "12V IN"
- board text added: "5V OUT"
- board text added: "BOOT"
- board text added: "DISPLAY"
- board text added: "DOWN"
- board text added: "EXT_LEDs"
- board text added: "GND 5V SIG"
- board text added: "GND TX RX 3V3"
- board text added: "GPS"
- board text added: "LEFT"
- board text added: "POWER"
- board text added: "RESET"
- board text added: "RIGHT"
- board text added: "SERVO"
- board text added: "STUDENTE: MATTIA FAIT ANNO ACCADEMICO: 2025/2026 CORSO: PROGETTAZIONE E PROTOTIPAZIONE DI SISTEMI ELETTRONICI UNIVERSITA' DI TRENTO"
- board text added: "UART"
- board text added: "UP"

Commit message: update
Parts:
- U2: value W25Q128JVE -> W25Q16JVUSSQ
- moved R14 16.9 mm to (152.8, 85.1)
- moved R13 16.5 mm to (151.2, 85.2), turned to -90 degrees
- moved C19 2.91 mm to (134.9, 65.9)
- moved C21 2.91 mm to (131.9, 67.4)
- moved C28 2.91 mm to (131.9, 65.9)
- moved C29 2.91 mm to (128.9, 67.4)
- moved C41 2.91 mm to (125.9, 67.4)
- moved C45 2.91 mm to (125.9, 65.9)
- moved C34 2.91 mm to (128.9, 65.9)
- moved C47 2.91 mm to (123.7, 66.6)
- moved BZ1 2.51 mm to (181.9, 79.5)
- moved NT1 1.07 mm to (146.5, 67.9), turned to -90 degrees
- moved D7 0.48 mm to (190.8, 104.5)
- moved D8 0.45 mm to (198.0, 104.5)
- moved D6 0.17 mm to (198.1, 98.6)
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Connections:
- net /power/POST_PPTC renamed Net-(D11-K)
- C42 pad 1: Net-(Q3-D) -> Net-(Q1-D)
- C44 pad 1: Net-(Q3-D) -> Net-(Q1-D)
Routing:
- net GND: track 0.00 -> 51.3 mm, vias 0 -> 39
- net /mcu/USB_DP: track 32.2 -> 11.4 mm, vias 2 -> 0
- net /mcu/USB_DN: track 32.0 -> 11.3 mm, vias 2 -> 0
- net /power/D-: track 66.6 -> 84.0 mm, vias 0 -> 2
- net /power/D+: track 68.7 -> 84.1 mm, vias 0 -> 2
- net /mcu/ESP-01_EN: track 71.8 -> 81.9 mm
- net +5V: track 263.0 -> 267.6 mm
- net /ui/BUTTON_R: track 62.8 -> 59.7 mm
- net Net-(BZ1--): track 25.3 -> 28.0 mm
- net /mcu/GPS_RST: track 48.3 -> 46.2 mm
- net Net-(R20-Pad2): track 114.7 -> 112.5 mm
- net /I2C0_SDA: track 86.9 -> 88.6 mm
- net Net-(D18-K): track 0.00 -> 1.69 mm
- net /mcu/UART0_RX: track 20.3 -> 21.4 mm
- net /sensors/UART_TX: track 84.3 -> 85.3 mm
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Other:
- board text added: "BUZZER"
- board text added: "DEBUG"
- board text added: "FLASH"
- board text added: "LED ALIVE"
- board text added: "MCU"
- board text added: "USB"

Commit message: update
Parts:
- added Q1: IRLML9301, Package_TO_SOT_SMD:SOT-23, F.Cu at (165.9, 111.6)
- U2: footprint Package_SON:WSON-8-1EP_8x6mm_P1.27mm_EP3.4x4.3mm -> Package_SO:SOIC-8_5.3x5.3mm_P1.27mm
- U5: value XC6705A331MR-G -> SC662k-3-3V; footprint Package_TO_SOT_SMD:SOT-23-5 -> Package_TO_SOT_SMD:SOT-23-5_HandSoldering
- U6: footprint Package_SO:SOIC-8_3.9x4.9mm_P1.27mm -> Package_TO_SOT_SMD:SOT-23-6
- moved C9 23.0 mm to (142.8, 102.2), turned to 180 degrees
- moved C15 16.8 mm to (152.0, 108.1)
- moved C17 12.0 mm to (147.1, 95.2), turned to 135 degrees
- moved C12 11.6 mm to (159.3, 102.1), turned to -45 degrees
- moved C10 8.48 mm to (152.0, 92.3)
- moved U10 6.13 mm to (167.4, 82.3)
- moved C13 4.99 mm to (156.6, 95.0), turned to 90 degrees
- moved C38 4.09 mm to (175.1, 89.5)
- moved D17 3.57 mm to (174.6, 87.8)
- moved C18 1.86 mm to (158.6, 97.3)
- moved U6 0.60 mm to (128.7, 87.7)
- moved C23 0.26 mm to (155.0, 114.1)
- moved U7 0.25 mm to (127.0, 129.3), turned to 0 degrees
- moved U2 0.20 mm to (140.2, 78.6)
- moved U5 0.19 mm to (133.2, 111.1)
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Connections:
- net Net-(D11-K) renamed /power/POST_PPTC
- net Net-(R6-Pad2) renamed /mcu/~{USB_BOOT}
- U7 pad 17: Net-(Q3-D) -> Net-(Q1-D)
- U7 pad 2: Net-(Q3-D) -> Net-(Q1-D)
- U7 pad 3: Net-(Q3-D) -> Net-(Q1-D)
Routing:
- net Net-(Q1-D): track 0.00 -> 70.8 mm, vias 0 -> 6
- net Net-(Q3-D): track 60.3 -> 0.00 mm
- net /sensors/UART_RX: track 79.9 -> 47.7 mm, vias 1 -> 2
- net /mcu/GPS_PPS: track 62.1 -> 81.1 mm, vias 4 -> 5
- net /mcu/LED_ALIVE: track 88.0 -> 72.3 mm, vias 2 -> 4
- net +3V3: track 335.1 -> 350.2 mm, vias 6 -> 8
- net GND: track 51.3 -> 59.1 mm, vias 39 -> 63
- net /sensors/UART_TX: track 85.3 -> 92.7 mm
- net Net-(U10-V_{OUT}): track 7.47 -> 14.1 mm
- net /mcu/GPS_EN: track 41.1 -> 46.0 mm
- net Net-(U6-VFB): track 58.2 -> 62.8 mm
- net +12V: track 27.2 -> 30.3 mm, vias 0 -> 2
- net /mcu/GPS_RST: track 46.2 -> 49.0 mm
- net /power/BUCK_VBST: track 5.42 -> 2.60 mm
- net /ui/BUTTON_U: track 49.3 -> 51.5 mm
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
Commit message: update
Parts:
- removed the Q3 at (166.8, 135.2)
- moved U9 3.54 mm to (161.2, 124.1)
- moved J2 1.70 mm to (157.3, 123.5)
- moved TP3 1.35 mm to (150.4, 65.5)
- moved C19 0.76 mm to (135.1, 66.6)
- moved C21 0.76 mm to (132.1, 68.1)
- moved C28 0.76 mm to (132.1, 66.6)
- moved C29 0.76 mm to (129.1, 68.1)
- moved C34 0.76 mm to (129.1, 66.6)
- moved C47 0.76 mm to (123.9, 67.4)
- moved C41 0.76 mm to (126.1, 68.1)
- moved C45 0.76 mm to (126.1, 66.6)
- moved C13 0.37 mm to (156.9, 94.8)
- moved C9 0.30 mm to (142.8, 102.5)
- moved R17 0.19 mm to (129.4, 119.8)
- turned C39 to 0 degrees
- renumbered Q1 to Q3
Connections:
- SW2 pad 2: /mcu/~{USB_BOOT} -> GND
- SW3 pad 2: /ui/BUTTON_U -> GND
- SW4 pad 2: /ui/BUTTON_L -> GND
- SW5 pad 2: /ui/BUTTON_R -> GND
- SW6 pad 2: /ui/BUTTON_D -> GND
Routing:
- net /power/VBUS: track 138.0 -> 77.2 mm, vias 0 -> 1
- net GND: track 59.1 -> 74.4 mm, vias 63 -> 95
- net /ui/BUTTON_R: track 61.3 -> 53.4 mm
- net /ui/BUTTON_U: track 51.5 -> 46.5 mm
- net /ui/BUTTON_L: track 46.7 -> 42.0 mm
- net /power/D-: track 84.0 -> 79.4 mm
- net /power/D+: track 84.1 -> 79.8 mm
- net /mcu/UART0_TX: track 26.1 -> 22.6 mm, vias 0 -> 1
- net /mcu/~{USB_BOOT}: track 16.2 -> 12.8 mm
- net Net-(R20-Pad2): track 111.8 -> 108.6 mm
- net /mcu/UART0_RX: track 20.3 -> 17.2 mm
- net Net-(U9-~{RST}): track 2.60 -> 4.73 mm
- net Net-(D7-DOUT): track 16.3 -> 18.2 mm
- net /sensors/UART_TX: track 92.7 -> 90.9 mm
- net +5V: track 267.6 -> 269.4 mm
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