File: hard/PSE.kicad_pcb (KiCad board)
At the start: 2 copper layers, 102.2 x 77.2 mm, 139 parts, among them J1 WS2812B, J10 SERVO_3, J2 Conn_01x03, J3 Vin, J4 USB_B_Mini, J5 Vout 5V, J6 I2C_3V3, J7 UART0_3V3, J8 SERVO_1, J9 SERVO_2, Q2 PDTC114YT, Q3 IRLML9301, Q4 IRLML9301, SW1 RESET_SW, SW2 PROG_SW, SW3 SW_U, SW4 SW_L, SW5 SW_R, SW6 SW_D, SW7 Power_button, U1 RP2040, U10 TC1047A, U2 W25Q16JVUSSQ, U3 AT24C256, U4 oled_0.96"_128x64px, U5 SC662k-3-3V, U6 TPS563201, U7 SAM-M8Q, U8 MMA8451Q, U9 ESP-01, Y1 12MHz

Commit message: update
Parts:
- moved C7 89.2 mm to (188.1, 77.6), turned to 0 degrees
- moved C5 88.0 mm to (188.1, 74.6)
- moved C8 87.9 mm to (188.1, 79.1)
- moved C6 86.6 mm to (188.1, 76.1), turned to 0 degrees
- moved C3 73.8 mm to (184.6, 94.4)
- moved C4 73.8 mm to (184.6, 92.9), turned to 180 degrees
- moved C2 70.0 mm to (184.6, 96.0)
- moved C1 70.0 mm to (184.6, 97.5), turned to 180 degrees
- moved C37 23.2 mm to (125.5, 115.6)
- moved C39 23.0 mm to (125.5, 117.6), turned to 180 degrees
- moved C40 10.9 mm to (116.3, 114.2), turned to -45 degrees
- moved C33 10.0 mm to (115.3, 115.3), turned to -45 degrees
- moved BZ1 8.80 mm to (174.9, 74.2)
- moved R24 0.64 mm to (163.6, 135.9)
Routing:
- net Net-(R20-Pad2): track 108.6 -> 77.0 mm, vias 0 -> 2
- net +3V3: track 350.8 -> 358.8 mm
- net Net-(BZ1--): track 28.0 -> 35.5 mm
- net GND: track 74.4 -> 68.3 mm, vias 95 -> 96
- net +5V: track 269.4 -> 267.7 mm
- net /mcu/PWM_SERVO1: track 53.0 -> 52.0 mm
- net /I2C0_SDA: track 85.7 -> 86.6 mm
- net Net-(U1-RUN): track 51.6 -> 50.9 mm
- net /mcu/GPS_EN: track 46.8 -> 47.5 mm
- net /sensors/UART_TX: track 90.9 -> 90.3 mm
Other:
- board text added: "MATTIA FAIT 2025/2026 PROGETTAZIONE E PROTOTIPAZIONE DI SISTEMI ELETTRONICI UNIVERSITA' DI TRENTO"
- board text removed: "STUDENTE: MATTIA FAIT ANNO ACCADEMICO: 2025/2026 CORSO: PROGETTAZIONE E PROTOTIPAZIONE DI SISTEMI ELETTRONICI UNIVERSITA' DI TRENTO"

Commit message: update
Parts:
- moved C19 37.4 mm to (161.2, 93.4), turned to 45 degrees
- moved C14 4.64 mm to (147.9, 82.8)
- moved C20 4.61 mm to (147.9, 84.3)
- moved C16 4.57 mm to (147.8, 81.3)
Routing:
- net +3V3: track 358.8 -> 363.2 mm
- net +1V1: track 41.5 -> 37.2 mm
- net GND: vias 96 -> 97

Commit message: update
Routing:
- net GND: track 68.3 -> 69.7 mm
- net /mcu/GPS_PPS: track 82.0 -> 83.2 mm
- net /sensors/UART_TX: track 90.3 -> 91.0 mm
Changed lines of the file:
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@@
 		(tags "resistor")
 		(property "Reference" "R13"
-			(at 0.1 1.49 90)
+			(at 1.49 1.47 90)
 			(layer "F.SilkS")
 			(effects
@@
 	)
 	(segment
+		(start 156.94 93.985)
+		(end 156.94 92.63)
+		(width 0.2)
+		(layer "F.Cu")
+		(net 3)
+	)
+	(segment
 		(start 140.411199 109.389799)
 		(end 140.439199 109.361799)
@@
 	)
 	(via
+		(at 120.56 124.08)
+		(size 0.5)
+		(drill 0.3)
+		(layers "F.Cu" "B.Cu")
+		(free yes)
+		(net 3)
+	)
+	(via
 		(at 136.17 76.71)
 		(size 0.5)
@@
 	)
 	(via
-		(at 127.08 130.09)
-		(size 0.5)
-		(drill 0.3)
-		(layers "F.Cu" "B.Cu")
-		(free yes)
-		(net 3)
-	)
-	(via
 		(at 149.26 134.45)
 		(size 0.5)
@@
 	)
 	(segment
-		(start 125.13 121.622)
-		(end 122.2045 121.622)
+		(start 121.69 123.85)
+		(end 121.84 124)
+		(width 0.2)
+		(layer "F.Cu")
+		(net 19)
+	)
+	(segment
+		(start 136.99 132.15)
+		(end 139 132.15)
+		(width 0.2)
+		(layer "F.Cu")
+		(net 19)
+	)
+	(segment
+		(start 132.4545 126.4805)
+		(end 132.502 126.528)
 		(width 0.2)
 		(layer "F.Cu")
@@
 	)
 	(segment
-		(start 146.16 99.3)
-		(end 146.309999 99.449999)
+		(start 122.2045 121.622)
+		(end 121.69 122.1365)
 		(width 0.2)
 		(layer "F.Cu")
@@
 	(segment
 		(start 132.502 127.192)
-		(end 131.8 127.894)
+		(end 132.19 127.504)
 		(width 0.2)
 		(layer "F.Cu")
@@
 	)
 	(segment
-		(start 125.13 120.84)
-		(end 125.13 121.622)
+		(start 132.502 134.373)
+		(end 134.767 134.373)
 		(width 0.2)
 		(layer "F.Cu")
@@
 	)
 	(segment
-		(start 136.99 132.15)
-		(end 139 132.15)
+		(start 146.16 99.3)
+		(end 146.309999 99.449999)
 		(width 0.2)
 		(layer "F.Cu")
@@
 	)
 	(segment
-		(start 125.1 120.81)
-		(end 125.13 120.84)
+		(start 132.19 134.061)
+		(end 132.502 134.373)
 		(width 0.2)
 		(layer "F.Cu")
@@
 	)
 	(segment
-		(start 121.69 122.1365)
-		(end 121.69 124.15)
+		(start 132.19 127.504)
+		(end 132.19 134.061)
 		(width 0.2)
 		(layer "F.Cu")
@@
 	)
 	(segment
-		(start 121.69 124.15)
-		(end 123.3 125.76)
+		(start 125.13 120.84)
+		(end 125.13 121.622)
 		(width 0.2)
 		(layer "F.Cu")
@@
 	)
 	(segment
-		(start 131.8 127.894)
-		(end 131.8 133.671)
+		(start 125.1 120.81)
+		(end 125.13 120.84)
 		(width 0.2)
 		(layer "F.Cu")
@@
 	)
 	(segment
-		(start 122.2045 121.622)
-		(end 121.69 122.1365)
+		(start 125.13 121.622)
+		(end 122.2045 121.622)
 		(width 0.2)
 		(layer "F.Cu")
@@
 	)
 	(segment
-		(start 131.8 133.671)
-		(end 132.502 134.373)
+		(start 132.4545 125.0445)
+		(end 132.4545 126.4805)
 		(width 0.2)
 		(layer "F.Cu")
@@
 	)
 	(segment
-		(start 123.3 125.76)
-		(end 131.07 125.76)
+		(start 121.69 122.1365)
+		(end 121.69 123.85)
 		(width 0.2)
 		(layer "F.Cu")
@@
 	)
 	(segment
-		(start 134.767 134.373)
-		(end 136.99 132.15)
+		(start 131.41 124)
+		(end 132.4545 125.0445)
 		(width 0.2)
 		(layer "F.Cu")
@@
 	)
 	(segment
-		(start 131.07 125.76)
+		(start 121.84 124)
+		(end 131.41 124)
+		(width 0.2)
+		(layer "F.Cu")
+		(net 19)
+	)
+	(segment
+		(start 132.502 126.528)
 		(end 132.502 127.192)
 		(width 0.2)
@@
 	)
 	(segment
-		(start 132.502 134.373)
-		(end 134.767 134.373)
+		(start 134.767 134.373)
+		(end 136.99 132.15)
 		(width 0.2)
 		(layer "F.Cu")
@@
 	)
 	(segment
-		(start 136.04 126.12)
-		(end 136.04 128.45)
-		(width 0.2)
-		(layer "F.Cu")
-		(net 32)
-	)
-	(segment
-		(start 140.203 131.703478)
-		(end 140.203 132.940522)
+		(start 132.366138 134.701)
+		(end 131.7605 135.306638)
 		(width 0.2)
 		(layer "F.Cu")
@@
 	)
 	(segment
-		(start 138.662 131.072)
-		(end 139.571522 131.072)
+		(start 164.21 108.87)
+		(end 162.63 108.87)
 		(width 0.2)
 		(layer "F.Cu")
@@
 	)
 	(segment
-		(start 164.21 108.87)
-		(end 162.63 108.87)
+		(start 139.571522 131.072)
+		(end 140.203 131.703478)
 		(width 0.2)
 		(layer "F.Cu")
@@
 	)
 	(segment
-		(start 136.04 128.45)
-		(end 138.662 131.072)
+		(start 136.04 126.12)
+		(end 136.04 128.45)
 		(width 0.2)
 		(layer "F.Cu")
@@
 	)
 	(segment
-		(start 125.0825 134.8745)
-		(end 125.0825 135.95)
+		(start 126.1965 137.27)
+		(end 125.0825 136.156)
 		(width 0.2)
 		(layer "F.Cu")
@@
 	)
 	(segment
-		(start 132.366138 134.701)
-		(end 131.835138 134.17)
+		(start 140.203 131.703478)
+		(end 140.203 132.940522)
 		(width 0.2)
 		(layer "F.Cu")
@@
 	)
 	(segment
-		(start 156.008995 102.249999)
-		(end 155.5475 102.249999)
+		(start 131.7605 135.306638)
+		(end 131.7605 137.078)
 		(width 0.2)
 		(layer "F.Cu")
@@
 	)
 	(segment
-		(start 139.571522 131.072)
-		(end 140.203 131.703478)
+		(start 136.04 128.45)
+		(end 138.662 131.072)
 		(width 0.2)
 		(layer "F.Cu")
@@
 	)
 	(segment
-		(start 131.835138 134.17)
-		(end 125.787 134.17)
+		(start 125.0825 136.156)
+		(end 125.0825 135.95)
 		(width 0.2)
 		(layer "F.Cu")
@@
 	)
 	(segment
-		(start 137.299478 134.701)
-		(end 132.366138 134.701)
+		(start 156.008995 102.249999)
+		(end 155.5475 102.249999)
+		(width 0.2)
+		(layer "F.Cu")
+		(net 32)
+	)
+	(segment
+		(start 131.5685 137.27)
+		(end 126.1965 137.27)
+		(width 0.2)
+		(layer "F.Cu")
+		(net 32)
+	)
+	(segment
+		(start 138.662 131.072)
+		(end 139.571522 131.072)
 		(width 0.2)
 		(layer "F.Cu")
@@
 	)
 	(segment
-		(start 125.787 134.17)
-		(end 125.0825 134.8745)
+		(start 137.299478 134.701)
+		(end 132.366138 134.701)
+		(width 0.2)
+		(layer "F.Cu")
+		(net 32)
+	)
+	(segment
+		(start 131.7605 137.078)
+		(end 131.5685 137.27)
 		(width 0.2)
 		(layer "F.Cu")
@@
 	)
 	(segment
-		(start 126.98 123.558862)
+		(start 126.702 121.848)
 		(end 126.702 123.280862)
 		(width 0.2)
@@
 	)
 	(segment
-		(start 126.98 124.14)
-		(end 126.98 123.558862)
+		(start 147.62 105.36)
+		(end 149.4725 103.5075)
 		(width 0.2)
 		(layer "F.Cu")
@@
 	)
 	(segment
-		(start 147.62 105.36)
-		(end 149.4725 103.5075)
+		(start 127.23 121.32)
+		(end 126.702 121.848)
 		(width 0.2)
 		(layer "F.Cu")
@@
 	)
 	(via
-		(at 126.98 124.14)
+		(at 127.23 121.32)
 		(size 0.5)
 		(drill 0.3)
@@
 	)
 	(segment
-		(start 140.559178 110.495)
-		(end 141.04 110.014178)
+		(start 141.04 110.014178)
+		(end 141.04 105.36)
 		(width 0.2)
 		(layer "B.Cu")
@@
 	)
 	(segment
-		(start 133.725 104.900822)
-		(end 134.510822 104.115)
+		(start 127.23 121.32)
+		(end 129.615 118.935)
 		(width 0.2)
 		(layer "B.Cu")
@@
 	)
 	(segment
-		(start 134.510822 104.115)
-		(end 134.929178 104.115)
+		(start 133.039178 118.935)
+		(end 133.725 118.249178)
 		(width 0.2)
 		(layer "B.Cu")
@@
 	)
 	(segment
-		(start 139.300822 110.495)
-		(end 140.559178 110.495)
+		(start 135.225 106.419178)
+		(end 139.300822 110.495)
 		(width 0.2)
 		(layer "B.Cu")
@@
 	)
 	(segment
-		(start 141.04 110.014178)
-		(end 141.04 105.36)
+		(start 134.510822 104.115)
+		(end 134.929178 104.115)
 		(width 0.2)
 		(layer "B.Cu")
@@
 	)
 	(segment
-		(start 127.834178 124.14)
-		(end 133.725 118.249178)
+		(start 133.725 104.900822)
+		(end 134.510822 104.115)
 		(width 0.2)
 		(layer "B.Cu")
@@
 	)
 	(segment
-		(start 126.98 124.14)
-		(end 127.834178 124.14)
+		(start 140.559178 110.495)
+		(end 141.04 110.014178)
 		(width 0.2)
 		(layer "B.Cu")
@@
 	)
 	(segment
-		(start 135.225 106.419178)
-		(end 139.300822 110.495)
+		(start 133.725 118.249178)
+		(end 133.725 104.900822)
 		(width 0.2)
 		(layer "B.Cu")
@@
 	)
 	(segment
-		(start 133.725 118.249178)
-		(end 133.725 104.900822)
+		(start 139.300822 110.495)
+		(end 140.559178 110.495)
+		(width 0.2)
+		(layer "B.Cu")
+		(net 47)
+	)
+	(segment
+		(start 129.615 118.935)
+		(end 133.039178 118.935)
 		(width 0.2)
 		(layer "B.Cu")
