File: hard/PSE.kicad_pcb (KiCad board)
At the start: 2 copper layers, 102.2 x 77.2 mm, 139 parts, among them J1 WS2812B, J10 SERVO_3, J2 Conn_01x03, J3 Vin, J4 USB_B_Mini, J5 Vout 5V, J6 I2C_3V3, J7 UART0_3V3, J8 SERVO_1, J9 SERVO_2, Q2 PDTC114YT, Q3 IRLML9301, Q4 IRLML9301, SW1 RESET_SW, SW2 PROG_SW, SW3 SW_U, SW4 SW_L, SW5 SW_R, SW6 SW_D, SW7 Power_button, U1 RP2040, U10 TC1047A, U2 W25Q16JVUSSQ, U3 AT24C256, U4 oled_0.96"_128x64px, U5 SC662k-3-3V, U6 TPS563201, U7 SAM-M8Q, U8 MMA8451Q, U9 ESP-01, Y1 12MHz

Commit message: correzione layout bottom
Routing:
- net /mcu/GPS_RST: track 48.8 -> 47.1 mm
