File: hard/power.kicad_sch (KiCad schematic)
At the start: 0 parts

Commit message: edit
Changed lines of the file:
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@@
 	)
 	(sheet
-		(at 33.02 62.23)
+		(at 64.77 106.045)
 		(size 22.86 13.97)
 		(exclude_from_sim no)
@@
 		)
 		(property "Sheetname" "bc"
-			(at 33.02 61.5184 0)
+			(at 64.77 105.3334 0)
 			(effects
 				(font
@@
 		)
 		(property "Sheetfile" "bc.kicad_sch"
-			(at 33.02 76.7846 0)
+			(at 64.77 120.5996 0)
 			(effects
 				(font

Commit message: update
Parts:
- added C30, C31: 10u, symbol Device:C
- added C32, C35, C38: 100n, symbol Device:C
- added C33, C34: 1u, symbol Device:C
- added C36, C37, C38: C, symbol Device:C
- added C6: 2.2u, symbol Device:C
- added D11: D_Zener, symbol Device:D_Zener
- added D12: S1B, symbol Device:D
- added D13, D19: RBR1VWM30ATFTR, symbol Device:D_Schottky_Small
- added D14, D15: 1N4148, symbol Device:D
- added D16: 3V3_LED, symbol Device:LED
- added D17: PDZ3.3B.115, symbol Device:D_Zener
- added D26: LED, symbol Device:LED
- added F1: 2016L05MR, symbol Device:Polyfuse
- added FB1: FerriteBead, symbol Device:FerriteBead
- added J3 (x2): Vin, symbol Connector:Screw_Terminal_01x02
- added J4: USB_B_Mini, symbol Connector:USB_B_Mini
- added L1: 2.2u, symbol Device:L
- added NT1: gnda-gnd, symbol Device:NetTie_2
- added Q4: IRLML9301, Package_TO_SOT_SMD:SOT-23, symbol Transistor_FET:IRLML9301
- added R15, R17, R29: 10k, symbol Device:R
- added R18: 1.8k, symbol Device:R
- added R19: 200, symbol Device:R
- added R20: 150k, symbol Device:R
- added R21: 56k, symbol Device:R
- added R22: 1k, symbol Device:R
- added R29: R, symbol Device:R
- added R30: 47k, symbol Device:R
- added R6, R7: 27, symbol Device:R
- added R9: 510, symbol Device:R
- added SW7: Power_button, symbol Switch:SW_Push
- added TP4: 3V3A, symbol Connector:TestPoint
- added U5: XC6705A331MR-G, Package_TO_SOT_SMD:SOT-23-5, symbol Regulator_Linear:XC6210B332MR
- added U6: TPS563201, Package_SO:SOIC-8_3.9x4.9mm_P1.27mm, symbol Regulator_Switching:XL1509-5.0
Connections:
- new net: D16.1 (K), R9.1
- new net: R20.2, R21.1, R22.1
- new net: D26.1 (K), R29.1
- new net: D15.2 (A), SW7.1
- new net: R17.2, R18.1, U6.4 (VFB)
- new net +12V: C30.1, C31.1, C32.1, D12.1 (K), SW7.2, U6.3 (VIN)
- new net +3V3: C34.1, D16.2 (A), R19.1, U5.5 (VOUT)
- new net +3V3A: C6.1, R19.2, TP4.1
- new net +5V: C33.1, C36.1, C37.1, C38.1, D13.1 (K), D19.2 (A), D26.2 (A), L1.2, Q4.2 (S), R17.1, R29.2, U5.1 (VIN), U5.3 (CE)
- new net 5V_EN: D14.2 (A)
- new net ANALOG_BATT: C38.1, D17.1 (K), R22.2
- new net BUCK_EN: D14.1 (K), D15.1 (K), R15.1, U6.5 (EN)
- new net BUCK_SW: C35.2, L1.1, U6.2 (SW)
- new net BUCK_VBST: C35.1, U6.6 (VBST)
- new net D+: J4.3 (D+), R6.1
- new net D-: J4.2 (D-), R7.2
- new net FILTERED_VBUS: D13.2 (A), FB1.1, Q4.3 (D)
- new net GND: C30.2, C31.2, C32.2, C33.2, C34.2, C36.2, C37.2, C38.2, C38.2, C6.2, D11.2 (A), D17.2 (A), J3.1 (Pin_1), J3.2 (Pin_2), J4.5 (GND), J4.6 (Shield), NT1.1, NT1.2, R15.2, R18.2, R21.2, R29.2, R30.2, R9.2, U5.2 (Vss), U6.1 (GND)
- new net OUTPUT_USB_EN: Q4.1 (G), R29.1
- new net POST_PPTC: D11.1 (K), D12.2 (A), F1.1, F1.2, J3.2 (Pin_2)
- new net USB_DN: R7.1
- new net USB_DP: R6.2
- new net USB_ID: J4.4 (ID), R30.1
- new net VBUS: FB1.2, J4.1 (VBUS)
- new net VOUT_5V: D19.1 (K), J3.1 (Pin_1)
Other:
- removed sheet bc
- removed sheet bcv
- removed sheet lvr
- removed sheet mini_usb
- note added: "Buck Converter: Vin 4.5-17V, Vout 3.3V 3A (max)"
- note added: "Mini USB"
- note added: "Poszionare vicino Rp2040"
- note added: "Regolatore di tensione lineare (LDO) 3.3V"
- note added: "Tensione di controllo Batteria"
- note added: "VIN"

Commit message: update
Parts:
- C37: renamed from C36; value C -> 22u
- C39: renamed from C37; value C -> 22u
- C40: renamed from C38; value C -> 100n
- D11: value D_Zener -> TVS VBR 17V IBR=1mA
- D18: renamed from D26; value LED -> 5V_LED
- J5: renamed from J3; value Vin -> Vout 5V
- R23: renamed from R29; value R -> 510
- renumbered C6 to C36, R6 to R13, R7 to R14, R9 to R16
Connections:
- net POST_PPTC: no longer F1.1, J3.2 (Pin_2)
- net VIN: now reaches R20.1
- net VIN: now also F1.1, J3.2 (Pin_2)
Other:
- note added: "1A trip"
- note removed: "VIN"
Changed lines of the file:
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@@
 		)
 	)
-	(text "VIN"
+	(text "1A trip"
 		(exclude_from_sim no)
-		(at 236.22 22.86 0)
+		(at 29.718 78.486 0)
 		(effects
 			(font
@@
 		)
 	)
+	(label "VIN"
+		(at 236.22 24.13 0)
+		(effects
+			(font
+				(size 1.27 1.27)
+			)
+			(justify left bottom)
+		)
+	)
 	(label "D+"
 		(at 34.29 38.1 0)
@@
 		)
 	)
-	(label "VIN"
+	(label "VIN_"
 		(at 34.29 74.93 0)
 		(effects
@@
 		)
 		(property "Netclass" "3V3"
-			(at 159.766 22.352 0)
+			(at 160.782 22.606 0)
 			(effects
 				(font
@@
 		)
 		(property "Netclass" "TP1"
-			(at 24.384 20.828 0)
+			(at 26.924 18.542 0)
 			(effects
 				(font
@@
 		)
 		(property "Component Class" "VBUS"
-			(at 22.86 23.114 0)
+			(at 26.416 21.082 0)
 			(effects
 				(font
@@
 		(dnp no)
 		(fields_autoplaced yes)
-		(property "Reference" "C38"
+		(property "Reference" "C40"
 			(at 182.88 77.4699 0)
 			(effects
@@
 			)
 		)
-		(property "Value" "C"
+		(property "Value" "100n"
 			(at 182.88 80.0099 0)
 			(effects
@@
 			(project "PSE"
 				(path "/13844229-b559-4868-a710-53f590233cb2/ca9a428d-b29f-459a-8b79-10121d41243b"
-					(reference "C38")
+					(reference "C40")
 					(unit 1)
 				)
@@
 		(on_board yes)
 		(dnp no)
-		(property "Reference" "R7"
+		(property "Reference" "R14"
 			(at 45.72 43.434 90)
 			(effects
@@
 			(project "PSE"
 				(path "/13844229-b559-4868-a710-53f590233cb2/ca9a428d-b29f-459a-8b79-10121d41243b"
-					(reference "R7")
+					(reference "R14")
 					(unit 1)
 				)
@@
 		(dnp no)
 		(fields_autoplaced yes)
-		(property "Reference" "R29"
+		(property "Reference" "R23"
 			(at 194.31 85.0899 0)
 			(effects
@@
 			)
 		)
-		(property "Value" "R"
+		(property "Value" "510"
 			(at 194.31 87.6299 0)
 			(effects
@@
 			(project "PSE"
 				(path "/13844229-b559-4868-a710-53f590233cb2/ca9a428d-b29f-459a-8b79-10121d41243b"
-					(reference "R29")
+					(reference "R23")
 					(unit 1)
 				)
@@
 		(dnp no)
 		(fields_autoplaced yes)
-		(property "Reference" "D26"
+		(property "Reference" "D18"
 			(at 195.58 79.0574 90)
 			(effects
@@
 			)
 		)
-		(property "Value" "LED"
+		(property "Value" "5V_LED"
 			(at 195.58 81.5974 90)
 			(effects
@@
 			(project "PSE"
 				(path "/13844229-b559-4868-a710-53f590233cb2/ca9a428d-b29f-459a-8b79-10121d41243b"
-					(reference "D26")
+					(reference "D18")
 					(unit 1)
 				)
@@
 		(on_board yes)
 		(dnp no)
-		(property "Reference" "R6"
+		(property "Reference" "R13"
 			(at 45.72 33.274 90)
 			(effects
@@
 			(project "PSE"
 				(path "/13844229-b559-4868-a710-53f590233cb2/ca9a428d-b29f-459a-8b79-10121d41243b"
-					(reference "R6")
+					(reference "R13")
 					(unit 1)
 				)
@@
 		(dnp no)
 		(fields_autoplaced yes)
-		(property "Reference" "C6"
+		(property "Reference" "C36"
 			(at 180.34 38.0999 0)
 			(effects
@@
 			(project "PSE"
 				(path "/13844229-b559-4868-a710-53f590233cb2/ca9a428d-b29f-459a-8b79-10121d41243b"
-					(reference "C6")
+					(reference "C36")
 					(unit 1)
 				)
@@
 		(dnp no)
 		(fields_autoplaced yes)
-		(property "Reference" "C37"
+		(property "Reference" "C39"
 			(at 172.72 77.4699 0)
 			(effects
@@
 			)
 		)
-		(property "Value" "C"
+		(property "Value" "22u"
 			(at 172.72 80.0099 0)
 			(effects
@@
 			(project "PSE"
 				(path "/13844229-b559-4868-a710-53f590233cb2/ca9a428d-b29f-459a-8b79-10121d41243b"
-					(reference "C37")
+					(reference "C39")
 					(unit 1)
 				)
@@
 		(dnp no)
 		(fields_autoplaced yes)
-		(property "Reference" "R9"
+		(property "Reference" "R16"
 			(at 161.29 38.0999 0)
 			(effects
@@
 			(project "PSE"
 				(path "/13844229-b559-4868-a710-53f590233cb2/ca9a428d-b29f-459a-8b79-10121d41243b"
-					(reference "R9")
+					(reference "R16")
 					(unit 1)
 				)
@@
 		(on_board yes)
 		(dnp no)
-		(fields_autoplaced yes)
 		(property "Reference" "D11"
 			(at 41.91 77.4699 90)
@@
 			)
 		)
-		(property "Value" "D_Zener"
-			(at 41.91 80.0099 90)
+		(property "Value" "TVS VBR 17V IBR=1mA"
+			(at 34.798 77.216 0)
 			(effects
 				(font
@@
 		(dnp no)
 		(fields_autoplaced yes)
-		(property "Reference" "C36"
+		(property "Reference" "C37"
 			(at 163.83 77.4699 0)
 			(effects
@@
 			)
 		)
-		(property "Value" "C"
+		(property "Value" "22u"
 			(at 163.83 80.0099 0)
 			(effects
@@
 			(project "PSE"
 				(path "/13844229-b559-4868-a710-53f590233cb2/ca9a428d-b29f-459a-8b79-10121d41243b"
-					(reference "C36")
+					(reference "C37")
 					(unit 1)
 				)
@@
 		(on_board yes)
 		(dnp no)
-		(fields_autoplaced yes)
-		(property "Reference" "J3"
-			(at 233.68 74.9299 0)
+		(property "Reference" "J5"
+			(at 229.87 67.564 0)
 			(effects
 				(font
@@
 			)
 		)
-		(property "Value" "Vin"
-			(at 233.68 77.4699 0)
+		(property "Value" "Vout 5V"
+			(at 228.092 70.358 0)
 			(effects
 				(font
@@
 			(project "PSE"
 				(path "/13844229-b559-4868-a710-53f590233cb2/ca9a428d-b29f-459a-8b79-10121d41243b"
-					(reference "J3")
+					(reference "J5")
 					(unit 1)
 				)

Commit message: update
Parts:
- C30, C31, C32, C33, C34, C35, C36, C37, C38, C39, C40: footprint (none) -> Capacitor_Tantalum_SMD:CP_EIA-1608-08_AVX-J
- D11, D12: footprint (none) -> Diode_SMD:D_SMA
- D13, D14, D19: footprint (none) -> Diode_SMD:D_SOD-123
- D15: footprint (none) -> Diode_SMD:D_SOD-123F
- D16: footprint (none) -> LED_SMD:LED_0805_2012Metric
- D17: footprint (none) -> Diode_SMD:D_SOD-323_HandSoldering
- D18: footprint (none) -> LED_SMD:LED_0805_2012Metric_Pad1.15x1.40mm_HandSolder
- F1: footprint (none) -> Fuse:Fuse_1206_3216Metric
- FB1: footprint (none) -> Capacitor_SMD:C_0805_2012Metric
- J4: footprint (none) -> Connector_USB:USB_Mini-B_Wuerth_65100516121_Horizontal
- L1: footprint (none) -> Capacitor_SMD:C_0603_1608Metric
- R13, R14, R15, R16, R17, R18, R19, R20, R21, R22, R23, R29, R30: footprint (none) -> Resistor_SMD:R_0201_0603Metric
- SW7: footprint (none) -> Button_Switch_SMD:Nidec_Copal_CAS-120A
- TP4: footprint (none) -> TestPoint:TestPoint_THTPad_D1.5mm_Drill0.7mm
Changed lines of the file:
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@@
 		)
 		(property "Netclass" "TP2"
-			(at 112.776 22.098 0)
+			(at 112.522 21.59 0)
 			(effects
 				(font
@@
 			)
 		)
-		(property "Footprint" ""
+		(property "Footprint" "Diode_SMD:D_SOD-123"
 			(at 77.47 25.4 90)
 			(effects
@@
 			)
 		)
-		(property "Footprint" ""
+		(property "Footprint" "Capacitor_Tantalum_SMD:CP_EIA-1608-08_AVX-J"
 			(at 180.0352 82.55 0)
 			(effects
@@
 			)
 		)
-		(property "Footprint" ""
+		(property "Footprint" "Resistor_SMD:R_0201_0603Metric"
 			(at 94.742 83.82 90)
 			(effects
@@
 			)
 		)
-		(property "Footprint" ""
+		(property "Footprint" "Resistor_SMD:R_0201_0603Metric"
 			(at 45.72 38.862 90)
 			(effects
@@
 			)
 		)
-		(property "Footprint" ""
+		(property "Footprint" "Capacitor_Tantalum_SMD:CP_EIA-1608-08_AVX-J"
 			(at 59.3852 82.55 0)
 			(effects
@@
 			)
 		)
-		(property "Footprint" ""
+		(property "Footprint" "LED_SMD:LED_0805_2012Metric"
 			(at 158.75 31.75 0)
 			(effects
@@
 			)
 		)
-		(property "Footprint" ""
-			(at 25.4 39.37 0)
+		(property "Footprint" "Connector_USB:USB_Mini-B_Wuerth_65100516121_Horizontal"
+			(at 5.334 38.1 90)
 			(effects
 				(font
 					(size 1.27 1.27)
 				)
-				(hide yes)
 			)
 		)
@@
 			)
 		)
-		(property "Footprint" ""
+		(property "Footprint" "TestPoint:TestPoint_THTPad_D1.5mm_Drill0.7mm"
 			(at 196.85 40.64 0)
 			(effects
@@
 			)
 		)
-		(property "Footprint" ""
+		(property "Footprint" "Capacitor_SMD:C_0805_2012Metric"
 			(at 48.26 23.622 90)
 			(effects
@@
 			)
 		)
-		(property "Footprint" ""
+		(property "Footprint" "Diode_SMD:D_SMA"
 			(at 54.61 74.93 0)
 			(effects
@@
 			)
 		)
-		(property "Footprint" ""
+		(property "Footprint" "Resistor_SMD:R_0201_0603Metric"
 			(at 27.432 46.99 90)
 			(effects
@@
 			)
 		)
-		(property "Footprint" ""
+		(property "Footprint" "Resistor_SMD:R_0201_0603Metric"
 			(at 241.3 37.338 90)
 			(effects
@@
 			)
 		)
-		(property "Footprint" ""
+		(property "Footprint" "Resistor_SMD:R_0201_0603Metric"
 			(at 189.992 86.36 90)
 			(effects
@@
 			)
 		)
-		(property "Footprint" ""
+		(property "Footprint" "Capacitor_Tantalum_SMD:CP_EIA-1608-08_AVX-J"
 			(at 69.5452 82.55 0)
 			(effects
@@
 			)
 		)
-		(property "Footprint" ""
+		(property "Footprint" "LED_SMD:LED_0805_2012Metric_Pad1.15x1.40mm_HandSolder"
 			(at 191.77 78.74 0)
 			(effects
@@
 			)
 		)
-		(property "Footprint" ""
+		(property "Footprint" "Resistor_SMD:R_0201_0603Metric"
 			(at 45.72 39.878 90)
 			(effects
@@
 			)
 		)
-		(property "Footprint" ""
+		(property "Footprint" "Button_Switch_SMD:Nidec_Copal_CAS-120A"
 			(at 81.28 109.22 0)
 			(effects
@@
 			)
 		)
-		(property "Footprint" ""
+		(property "Footprint" "Resistor_SMD:R_0201_0603Metric"
 			(at 234.442 31.75 90)
 			(effects
@@
 			)
 		)
-		(property "Footprint" ""
+		(property "Footprint" "Capacitor_Tantalum_SMD:CP_EIA-1608-08_AVX-J"
 			(at 111.4552 35.56 0)
 			(effects
@@
 			)
 		)
-		(property "Footprint" ""
+		(property "Footprint" "Capacitor_Tantalum_SMD:CP_EIA-1608-08_AVX-J"
 			(at 136.1948 74.93 0)
 			(effects
@@
 			)
 		)
-		(property "Footprint" ""
+		(property "Footprint" "Diode_SMD:D_SOD-323_HandSoldering"
 			(at 256.54 39.37 0)
 			(effects
@@
 			)
 		)
-		(property "Footprint" ""
+		(property "Footprint" "Diode_SMD:D_SOD-123"
 			(at 87.63 93.98 0)
 			(effects
@@
 			)
 		)
-		(property "Footprint" ""
+		(property "Footprint" "Capacitor_Tantalum_SMD:CP_EIA-1608-08_AVX-J"
 			(at 177.4952 43.18 0)
 			(effects
@@
 			)
 		)
-		(property "Footprint" ""
+		(property "Footprint" "Diode_SMD:D_SOD-123"
 			(at 210.82 74.93 90)
 			(effects
@@
 			)
 		)
-		(property "Footprint" ""
+		(property "Footprint" "Capacitor_Tantalum_SMD:CP_EIA-1608-08_AVX-J"
 			(at 144.4752 35.56 0)
 			(effects
@@
 			)
 		)
-		(property "Footprint" ""
+		(property "Footprint" "Resistor_SMD:R_0201_0603Metric"
 			(at 82.55 46.228 90)
 			(effects
@@
 			)
 		)
-		(property "Footprint" ""
+		(property "Footprint" "Capacitor_Tantalum_SMD:CP_EIA-1608-08_AVX-J"
 			(at 169.8752 82.55 0)
 			(effects
@@
 			)
 		)
-		(property "Footprint" ""
+		(property "Footprint" "Fuse:Fuse_1206_3216Metric"
 			(at 35.56 73.66 0)
 			(effects
@@
 			)
 		)
-		(property "Footprint" ""
+		(property "Footprint" "Capacitor_SMD:C_0603_1608Metric"
 			(at 143.51 74.93 0)
 			(effects
@@
 			)
 		)
-		(property "Footprint" ""
+		(property "Footprint" "Resistor_SMD:R_0201_0603Metric"
 			(at 156.972 39.37 90)
 			(effects
@@
 			)
 		)
-		(property "Footprint" ""
+		(property "Footprint" "Capacitor_Tantalum_SMD:CP_EIA-1608-08_AVX-J"
 			(at 80.9752 82.55 0)
 			(effects
@@
 			)
 		)
-		(property "Footprint" ""
+		(property "Footprint" "Resistor_SMD:R_0201_0603Metric"
 			(at 174.752 31.75 90)
 			(effects
@@
 			)
 		)
-		(property "Footprint" ""
+		(property "Footprint" "Resistor_SMD:R_0201_0603Metric"
 			(at 146.812 88.9 90)
 			(effects
@@
 			)
 		)
-		(property "Footprint" ""
+		(property "Footprint" "Diode_SMD:D_SMA"
 			(at 39.37 78.74 0)
 			(effects
@@
 			)
 		)
-		(property "Footprint" ""
+		(property "Footprint" "Diode_SMD:D_SOD-123F"
 			(at 87.63 104.14 0)
 			(effects
@@
 			)
 		)
-		(property "Footprint" ""
+		(property "Footprint" "Capacitor_Tantalum_SMD:CP_EIA-1608-08_AVX-J"
 			(at 160.9852 82.55 0)
 			(effects
@@
 			)
 		)
-		(property "Footprint" ""
+		(property "Footprint" "Capacitor_Tantalum_SMD:CP_EIA-1608-08_AVX-J"
 			(at 246.0752 43.18 0)
 			(effects
@@
 			)
 		)
-		(property "Footprint" ""
+		(property "Footprint" "Resistor_SMD:R_0201_0603Metric"
 			(at 234.442 39.37 90)
 			(effects
@@
 			)
 		)
-		(property "Footprint" ""
+		(property "Footprint" "Resistor_SMD:R_0201_0603Metric"
 			(at 146.812 78.74 90)
 			(effects

Commit message: update
Changed lines of the file:
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@@
 			(font
 				(size 1.27 1.27)
-				(thickness 0.254)
-				(bold yes)
+				(thickness 0.1588)
 			)
 			(justify left bottom)
@@
 			(font
 				(size 1.27 1.27)
-				(thickness 0.254)
-				(bold yes)
+				(thickness 0.1588)
 			)
 			(justify left bottom)
@@
 			(font
 				(size 1.27 1.27)
-				(thickness 0.254)
-				(bold yes)
+				(thickness 0.1588)
 			)
 			(justify left bottom)
@@
 			(font
 				(size 1.27 1.27)
-				(thickness 0.254)
-				(bold yes)
+				(thickness 0.1588)
 			)
 			(justify left bottom)
@@
 		(shape round)
 		(at 29.21 25.4 0)
+		(fields_autoplaced yes)
 		(effects
 			(font
@@
 		)
 		(property "Netclass" "TP1"
-			(at 26.924 18.542 0)
+			(at 29.9085 22.86 0)
 			(effects
 				(font
@@
 		)
 		(property "Component Class" "VBUS"
-			(at 26.416 21.082 0)
+			(at 29.9085 24.3205 0)
 			(effects
 				(font
@@
 					(size 1.27 1.27)
 				)
-			)
-		)
+				(hide yes)
+			)
+		)

Commit message: update
Connections:
- net +3V3A renamed +3.3VA
Changed lines of the file:
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@@
 	(wire
 		(pts
+			(xy 58.42 72.39) (xy 58.42 74.93)
+		)
+		(stroke
+			(width 0)
+			(type default)
+		)
+	)
+	(wire
+		(pts
 			(xy 121.92 77.47) (xy 133.35 77.47)
 		)
@@
 			(justify left bottom)
 		)
-		(property "Netclass" "TP2"
+		(property "Netclass" "5V"
 			(at 112.522 21.59 0)
 			(effects
@@
 			)
 		)
-		(property "Component Class" "5V"
+		(property "Component Class" "TP2"
 			(at 113.03 23.876 0)
 			(effects
@@
 		(shape round)
 		(at 29.21 25.4 0)
-		(fields_autoplaced yes)
 		(effects
 			(font
@@
 			(justify left bottom)
 		)
-		(property "Netclass" "TP1"
-			(at 29.9085 22.86 0)
+		(property "Netclass" "VBUS"
+			(at 29.972 20.828 0)
 			(effects
 				(font
@@
 			)
 		)
-		(property "Component Class" "VBUS"
-			(at 29.9085 24.3205 0)
+		(property "Component Class" "TP1"
+			(at 29.972 23.876 0)
 			(effects
 				(font
@@
 	)
 	(symbol
+		(lib_name "VD_1")
 		(lib_id "power:VD")
 		(at 196.85 35.56 0)
@@
 			)
 		)
-		(property "Value" "+3V3A"
+		(property "Value" "+3.3VA"
 			(at 197.358 31.496 0)
 			(effects
@@
 		(dnp no)
 		(property "Reference" "TP4"
-			(at 197.612 38.608 90)
+			(at 197.612 38.354 90)
 			(effects
 				(font
@@
 		)
 		(property "Value" "3V3A"
-			(at 196.596 40.64 90)
+			(at 196.85 40.64 90)
 			(effects
 				(font
@@
 	)
 	(symbol
+		(lib_name "PWR_FLAG_1")
 		(lib_id "power:PWR_FLAG")
 		(at 187.96 35.56 0)
@@
 	(symbol
 		(lib_id "power:VCC")
-		(at 58.42 74.93 0)
+		(at 58.42 72.39 0)
 		(unit 1)
 		(exclude_from_sim no)
@@
 		(dnp no)
 		(property "Reference" "#PWR048"
-			(at 58.42 78.74 0)
+			(at 58.42 76.2 0)
 			(effects
 				(font
@@
 		)
 		(property "Value" "+12V"
-			(at 60.452 71.374 0)
+			(at 60.452 68.834 0)
 			(effects
 				(font
@@
 		)
 		(property "Footprint" ""
-			(at 58.42 74.93 0)
+			(at 58.42 72.39 0)
 			(effects
 				(font
@@
 		)
 		(property "Datasheet" ""
-			(at 58.42 74.93 0)
+			(at 58.42 72.39 0)
 			(effects
 				(font
@@
 		)
 		(property "Description" "Power symbol creates a global label with name \"VCC\""
-			(at 58.42 74.93 0)
+			(at 58.42 72.39 0)
 			(effects
 				(font

Commit message: update
Parts:
- added TP1: VBUS, TestPoint:TestPoint_THTPad_D1.5mm_Drill0.7mm, symbol Connector:TestPoint
- added TP2: 5V, TestPoint:TestPoint_THTPad_D1.5mm_Drill0.7mm, symbol Connector:TestPoint
- added TP3: 3V3, TestPoint:TestPoint_THTPad_D1.5mm_Drill0.7mm, symbol Connector:TestPoint
- C30, C31, C37, C39: footprint Capacitor_Tantalum_SMD:CP_EIA-1608-08_AVX-J -> Capacitor_SMD:C_0805_2012Metric
- C32, C33, C34, C35, C36, C38, C40: footprint Capacitor_Tantalum_SMD:CP_EIA-1608-08_AVX-J -> Capacitor_SMD:C_0603_1608Metric
- D15: footprint Diode_SMD:D_SOD-123F -> Diode_SMD:D_SOD-123
- D18: footprint LED_SMD:LED_0805_2012Metric_Pad1.15x1.40mm_HandSolder -> LED_SMD:LED_0805_2012Metric
- J3, J5: footprint (none) -> libs:TerminalBlock_bornier-2_P5.08mm
- NT1: footprint (none) -> NetTie:NetTie-2_SMD_Pad0.5mm
- R13, R14, R15, R16, R17, R18, R19, R20, R21, R22, R23, R29, R30: footprint Resistor_SMD:R_0201_0603Metric -> Resistor_SMD:R_0603_1608Metric
- SW7: footprint Button_Switch_SMD:Nidec_Copal_CAS-120A -> Button_Switch_SMD:SW_SPST_EVQP0
Connections:
- net +3V3: now also TP3.1
- net +5V: now also TP2.1
- net VBUS: now also TP1.1

Commit message: update
Parts:
- removed U5: XC6705A331MR-G, Package_TO_SOT_SMD:SOT-23-5, symbol Regulator_Linear:XC6210B332MR
- removed U6: TPS563201, Package_SO:SOIC-8_3.9x4.9mm_P1.27mm, symbol Regulator_Switching:XL1509-5.0
- added U5: XC6705A331MR-G, Package_TO_SOT_SMD:SOT-23-5, symbol libs:XC6210B332MR
- added U6: TPS563201, Package_SO:SOIC-8_3.9x4.9mm_P1.27mm, symbol libs:XL1509-5.0
Connections:
- net +12V: now also U6.3 (VIN)
- net +3V3: now also U5.5 (VOUT)
- net +5V: now also U5.1 (VIN), U5.3 (CE)
- net BUCK_EN: now also U6.5 (EN)
- net BUCK_SW: now also U6.2 (SW)
- net BUCK_VBST: now also U6.6 (VBST)
- net GND: now also U5.2 (Vss), U6.1 (GND)
- net at R17.2, R18.1: now also U6.4 (VFB)
- net POST_PPTC: no longer names the net of D11.1 (K), D12.2 (A), F1.2
Other:
- note added: "BUCK_VIN"
- note added: "POST_PPTC"
- note added: "VIN_"
