File: hard/power.kicad_sch (KiCad schematic)
At the start: 48 parts, among them J3 Vin, J4 USB_B_Mini, J5 Vout 5V, Q4 IRLML9301, SW7 Power_button, U5 XC6705A331MR-G, U6 TPS563201

Commit message: update
Parts:
- U5: value XC6705A331MR-G -> SC662k-3-3V; footprint Package_TO_SOT_SMD:SOT-23-5 -> Package_TO_SOT_SMD:SOT-23-5_HandSoldering
- U6: footprint Package_SO:SOIC-8_3.9x4.9mm_P1.27mm -> Package_TO_SOT_SMD:SOT-23-6
Connections:
- net POST_PPTC: now reaches D11.1 (K), D12.2 (A), F1.2
Other:
- note added: "NOTA: posizionare induttore e condensatori filtro passa basso vicino a SW"
- note removed: "BUCK_VIN"
- note removed: "POST_PPTC"
- note removed: "VIN_"
- company: (none) -> UNITN - DISI
- title: (none) -> Sezione di Alimentazione
- moved on the sheet: C30, C31, C32, C33, C34, C35, C36, C37, C38, C39, C40, D11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
