File: hard/PSE.kicad_sch (KiCad schematic)
At the start: 0 parts

Commit message: edit
Other:
- company: (none) -> Universita' di Trento
- title: (none) -> PSE
Changed lines of the file:
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@@
 	(generator_version "9.0")
 	(paper "A4")
-	(sheet
-		(at 67.31 57.15)
+	(title_block
+		(title "PSE")
+		(company "Universita' di Trento")
+	)
+	(sheet
+		(at 118.11 117.475)
 		(size 29.21 15.24)
 		(exclude_from_sim no)
@@
 		)
 		(property "Sheetname" "led"
-			(at 67.31 56.4384 0)
+			(at 118.11 116.7634 0)
 			(effects
 				(font
@@
 		)
 		(property "Sheetfile" "led.kicad_sch"
-			(at 67.31 72.9746 0)
+			(at 118.11 133.2996 0)
 			(effects
 				(font
@@
 	)
 	(sheet
-		(at 19.05 54.61)
+		(at 38.1 127)
 		(size 29.21 24.13)
 		(exclude_from_sim no)
@@
 		)
 		(property "Sheetname" "mem"
-			(at 19.05 53.8984 0)
+			(at 38.1 126.2884 0)
 			(effects
 				(font
@@
 		)
 		(property "Sheetfile" "mem.kicad_sch"
-			(at 19.05 79.3246 0)
+			(at 38.1 151.7146 0)
 			(effects
 				(font
@@
 	)
 	(sheet
-		(at 146.05 20.32)
+		(at 226.06 46.99)
 		(size 39.37 27.94)
 		(exclude_from_sim no)
@@
 		)
 		(property "Sheetname" "ui"
-			(at 146.05 19.6084 0)
+			(at 226.06 46.2784 0)
 			(effects
 				(font
@@
 		)
 		(property "Sheetfile" "ui.kicad_sch"
-			(at 146.05 48.8446 0)
+			(at 226.06 75.5146 0)
 			(effects
 				(font
@@
 	)
 	(sheet
-		(at 72.39 20.32)
+		(at 152.4 46.99)
 		(size 49.53 24.13)
 		(exclude_from_sim no)
@@
 		)
 		(property "Sheetname" "mcu"
-			(at 72.39 19.6084 0)
+			(at 152.4 46.2784 0)
 			(effects
 				(font
@@
 		)
 		(property "Sheetfile" "mcu.kicad_sch"
-			(at 72.39 45.0346 0)
+			(at 152.4 71.7046 0)
 			(effects
 				(font
@@
 		)
 		(property "Field2" ""
-			(at 72.39 20.32 0)
+			(at 152.4 46.99 0)
 			(effects
 				(font
@@
 	)
 	(sheet
-		(at 121.92 58.42)
+		(at 187.96 113.665)
 		(size 36.83 19.05)
 		(exclude_from_sim no)
@@
 		)
 		(property "Sheetname" "sensors"
-			(at 121.92 57.7084 0)
+			(at 187.96 112.9534 0)
 			(effects
 				(font
@@
 		)
 		(property "Sheetfile" "sensors.kicad_sch"
-			(at 121.92 78.0546 0)
+			(at 187.96 133.2996 0)
 			(effects
 				(font
@@
 	)
 	(sheet
-		(at 17.78 16.51)
-		(size 38.1 29.21)
+		(at 41.275 43.815)
+		(size 52.705 36.195)
 		(exclude_from_sim no)
 		(in_bom yes)
@@
 		)
 		(property "Sheetname" "power"
-			(at 17.78 15.7984 0)
+			(at 41.275 43.1034 0)
 			(effects
 				(font
@@
 		)
 		(property "Sheetfile" "power.kicad_sch"
-			(at 17.78 46.3046 0)
-			(effects
-				(font
+			(at 41.275 80.5946 0)
+			(effects
+				(font

Commit message: update
Other:
- removed sheet mem
- sheet led ports: added DIN; removed none
- sheet mcu ports: added 5V_EN, BUZZER_PWM, ESP-01_EN, GPS_EN, GPS_PPS, GPS_RST, I2CO_SCL, I2CO_SDA, INT1_ACC, INT2_ACC, LED_ALIVE, OUTPUT_USBEN, PWM_SERVO1, PWM_SERVO2, PWM_SERVO3, RGB_LED, SW_DOWN, SW_LEFT, SW_RIGHT, SW_UP, TEMP_SENS, UART0_RX, UART0_TX, UART1_RX, UART1_TX, USB_DN, USB_DP, USB_ID, VBAT; removed none
- sheet power ports: added 5V_EN, ANALOG_BATT, OUTPUT_USB_EN, USB_DN, USB_DP, USB_ID; removed none
- sheet sensors ports: added ACC_INT1, ACC_INT2, ACC_SCL, ACC_SDA, ESP_EN, ESP_RX, ESP_TX, EXT_I2C_SCL, EXT_I2C_SDA, RX_SAM, SAM_EN, SAM_PPS, SAM_RST, SERVO_1, SERVO_2, SERVO_3, TEMP, TX_SAM; removed none
- sheet ui ports: added BUZZER, LED_ALIVE, SCL_DISPLAY, SDA_DISPLAY, SW_DOWN, SW_LEFT, SW_RIGHT, SW_UP; removed none
- note added: "I2C0_SCL"
- note added: "I2C0_SDA"

Commit message: update
Other:
- note removed: "I2C0_SCL"
- note removed: "I2C0_SDA"

Commit message: update
Other:
- sheet mcu ports: added I2C0_SCL, I2C0_SDA; removed I2CO_SCL, I2CO_SDA
Changed lines of the file:
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@@
 			)
 		)
-		(pin "I2CO_SCL" output
+		(pin "I2C0_SCL" output
 			(at 162.56 106.68 0)
 			(effects
@@
 			)
 		)
-		(pin "I2CO_SDA" output
+		(pin "I2C0_SDA" output
 			(at 162.56 104.14 0)
 			(effects

Commit message: update
Changed lines of the file:
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@@
+		)
+	)
+	(label "I2C0_SDA"
+		(at 175.26 104.14 180)
+		(effects
+			(font
+				(size 1.27 1.27)
+			)
+			(justify right bottom)
 		)
 	)
@@
 		(effects
 			(font
+				(size 1.27 1.27)
+			)
+			(justify right bottom)
+		)
+	)
+	(label "I2C0_SCL"
+		(at 175.26 106.68 180)
+		(effects
+			(font

Commit message: update
Parts:
- added H1, H2, H3, H4: MountingHole, MountingHole:MountingHole_3.2mm_M3_Pad_Via, symbol Mechanical:MountingHole
Other:
- note added: "Fori di Montaggio"

Commit message: update
Other:
- note added: "Schematico principale di Progetto"
- company: Universita' di Trento -> Universita' di Trento - DISI
- title: PSE -> Progettazione e Prototipazione di Sistemi Elettronici
- moved on the sheet: H1, H2, H3, H4
