File: hard/mcu.kicad_sch (KiCad schematic)
At the start: 0 parts

Commit message: update
Parts:
- added C1, C2, C39, C40, C41, C42, C43, C44, C45: C, symbol Device:C
- added C14, C15: 2.2u, symbol Device:C
- added C16, C17, C18: 100n, symbol Device:C
- added C21: DNP 100n, symbol Device:C
- added J2: Conn_01x03, symbol Connector_Generic:Conn_01x03
- added R1: R, symbol Device:R
- added R12, R5: 10k, symbol Device:R
- added R6: 1k, symbol Device:R
- added SW2: PROG_SW, symbol Switch:SW_MEC_5G
- added SW6: RESET_SW, symbol Switch:SW_Push
- added U1: AT24C256, Package_SO:SOIC-8_3.9x4.9mm_P1.27mm, symbol Memory_EEPROM:AT24CS01-SSHM
- added U1: RP2040, Package_DFN_QFN:QFN-56-1EP_7x7mm_P0.4mm_EP3.2x3.2mm, symbol MCU_RaspberryPi:RP2040
- added U2: W25Q128JVE, Package_SON:WSON-8-1EP_8x6mm_P1.27mm_EP3.4x4.3mm, symbol Memory_Flash:W25Q128JVE
- added Y1: 12MHz, symbol Device:Crystal_GND23
Connections:
- new net: C2.1, Y1.1
- new net: C1.1, R1.2, Y1.4
- new net: C18.1, R12.2, SW6.2, U1.26 (RUN)
- new net: R5.2, R6.1, U2.1 (~{CS})
- new net: R6.2, SW2.1 (A), SW2.2 (A)
- new net +1V1: C14.1, C16.1, C17.1, U1.23 (DVDD), U1.45 (VREG_VOUT), U1.50 (DVDD)
- new net +3.3VA: U1.43 (ADC_AVDD)
- new net +3V3: C15.1, C21.1, C39.1, C40.1, C41.1, C42.1, C43.1, C44.1, C45.1, R12.1, R5.1, U1.1 (IOVDD), U1.10 (IOVDD), U1.22 (IOVDD), U1.33 (IOVDD), U1.42 (IOVDD), U1.44 (VREG_IN), U1.48 (USB_VDD), U1.49 (IOVDD), U1.8 (VCC), U2.8 (VCC)
- new net 5V_EN: U1.14 (GPIO11)
- new net BUZZER_PWM: U1.32 (GPIO21)
- new net ESP-01_EN: U1.5 (GPIO3)
- new net GND: C1.2, C14.2, C15.2, C16.2, C17.2, C18.2, C2.2, C21.2, C39.2, C40.2, C41.2, C42.2, C43.2, C44.2, C45.2, J2.2 (Pin_2), SW2.3 (B), SW2.4 (B), SW6.1, U1.1 (A0), U1.19 (TESTEN), U1.2 (A1), U1.4 (GND), U1.57 (GND), U1.7 (WP), U2.4 (GND), Y1.2, Y1.3
- new net GPS_EN: U1.29 (GPIO18)
- new net GPS_PPS: U1.30 (GPIO19)
- new net GPS_RST: U1.15 (GPIO12)
- new net I2CO_SCL: U1.3 (GPIO1)
- new net I2CO_SDA: U1.2 (GPIO0)
- new net INT1_ACC: U1.17 (GPIO14)
- new net INT2_ACC: U1.18 (GPIO15)
- new net LED_ALIVE: U1.31 (GPIO20)
- new net OUTPUT_USBEN: U1.39 (GPIO27/ADC1)
- new net PWM_SERVO1: U1.11 (GPIO8)
- new net PWM_SERVO2: U1.12 (GPIO9)
- new net PWM_SERVO3: U1.9 (GPIO7)
- new net RGB_LED: U1.16 (GPIO13)
- new net SW_DOWN: U1.35 (GPIO23)
- new net SW_LEFT: U1.37 (GPIO25)
- new net SW_RIGHT: U1.36 (GPIO24)
- new net SW_UP: U1.34 (GPIO22)
- new net TEMP_SENS: U1.38 (GPIO26/ADC0)
- new net UART0_RX: U1.28 (GPIO17)
- new net UART0_TX: U1.27 (GPIO16)
- new net UART1_RX: U1.7 (GPIO5)
- new net UART1_TX: U1.6 (GPIO4)
- new net USB_DN: U1.46 (USB_DM)
- new net USB_DP: U1.47 (USB_DP)
- new net USB_ID: U1.4 (GPIO2)
- new net VBAT: U1.40 (GPIO28/ADC2)
- no-connect marks 0 -> 4
Other:
- note added: "12CO_SCL"
- note added: "Circuito Principale RP2040"
- note added: "Crystal"
- note added: "Debug"
- note added: "EEPROM"
- note added: "FLASH_CLK"
- note added: "FLASH_CS"
- note added: "FLASH_D0"
- note added: "FLASH_D1"
- note added: "FLASH_D2"
- note added: "FLASH_D3"
- note added: "Flash"
- note added: "I2CO_SCL"
- note added: "I2CO_SDA"
- note added: "NOTA: posizionare vicino i pin: IOVDD, USB_VDD"
- note added: "RUN"
- note added: "SWCLK"
- note added: "SWDIO"
- note added: "XIN"
- note added: "XOUT"
- note added: "~{FLASH_CS}"
- note added: "~{FLASH_D2}"
- note added: "~{USB_BOOT}"

Commit message: update
Parts:
- C10: renamed from C40; value C -> 100n
- C12: renamed from C41; value C -> 100n
- C13: renamed from C42; value C -> 100n
- C15: renamed from C43; value C -> 100n
- C17: renamed from C44; value C -> 100n
- C18: renamed from C45; value C -> 100n
- C22: renamed from C2; value C -> 18p
- C23: renamed from C1; value C -> 18p
- C9: renamed from C39; value C -> 100n
- renumbered C18 to C11, C17 to C14, C15 to C19, C14 to C20, R12 to R4, R1 to R7, SW6 to SW1, U1 to U3
Connections:
- net I2CO_SDA: now also U3.5 (SDA)
- net XIN: now reaches C22.1, Y1.1
- net XIN: now also U1.20 (XIN)
- net C_XOUT: now reaches C23.1, R7.2, Y1.4
- net FLASH_D1: now reaches U2.2 (DO_IO1)
- net FLASH_D1: now also U1.55 (QSPI_SD1)
- net ~{FLASH_D2}: now reaches U2.3 (WP_IO2)
- net FLASH_D0: now reaches U2.5 (DI_IOO)
- net FLASH_D0: now also U1.53 (QSPI_SD0)
- net FLASH_CLK: now reaches U2.6 (CLK)
- net FLASH_CLK: now also U1.52 (QSPI_SCLK)
- net FLASH_D3: now reaches U2.7 (HOLD_IO3)
- net FLASH_D3: now also U1.51 (QSPI_SD3)
- net SWDIO: now reaches J2.1 (Pin_1)
- net SWDIO: now also U1.25 (SWD)
- net SWCLK: now reaches J2.3 (Pin_3)
- net SWCLK: now also U1.24 (SWCLK)
- net XOUT: now reaches R7.1
- net XOUT: now also U1.21 (XOUT)
- net 12CO_SCL: now reaches U3.6 (SCL)
- net FLASH_D2: now reaches U1.54 (QSPI_SD2)
- net FLASH_CS: now reaches U1.56 (QSPI_SS)
Other:
- note removed: "12CO_SCL"
- note removed: "FLASH_CLK"
- note removed: "FLASH_CS"
- note removed: "FLASH_D0"
- note removed: "FLASH_D1"
- note removed: "FLASH_D2"
- note removed: "FLASH_D3"
- note removed: "SWCLK"
- note removed: "SWDIO"
- note removed: "XIN"
- note removed: "XOUT"
- note removed: "~{FLASH_D2}"

Commit message: update
Parts:
- C10, C11, C12, C13, C14, C15, C16, C17, C18, C19, C20, C21, C22, C23: footprint (none) -> Capacitor_Tantalum_SMD:CP_EIA-1608-08_AVX-J
- C9: footprint (none) -> Capacitor_Tantalum_SMD:CP_EIA-1608-10_AVX-L
- J2: footprint (none) -> Connector:BJB_Pico_46.110.1001_Receptacle_Horizontal
- R4, R5, R6, R7: footprint (none) -> Resistor_SMD:R_0201_0603Metric
- SW1, SW2: footprint (none) -> Button_Switch_SMD:Nidec_Copal_CAS-120A
- Y1: footprint (none) -> Crystal:Crystal_SMD_3225-4Pin_3.2x2.5mm_HandSoldering
Changed lines of the file:
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@@
 			)
 		)
-		(property "Footprint" ""
+		(property "Footprint" "Capacitor_Tantalum_SMD:CP_EIA-1608-08_AVX-J"
 			(at 77.1652 173.99 0)
 			(effects
@@
 			)
 		)
-		(property "Footprint" ""
+		(property "Footprint" "Capacitor_Tantalum_SMD:CP_EIA-1608-08_AVX-J"
 			(at 112.7252 173.99 0)
 			(effects
@@
 			)
 		)
-		(property "Footprint" ""
+		(property "Footprint" "Crystal:Crystal_SMD_3225-4Pin_3.2x2.5mm_HandSoldering"
 			(at 251.46 26.67 0)
 			(effects
@@
 			)
 		)
-		(property "Footprint" ""
+		(property "Footprint" "Capacitor_Tantalum_SMD:CP_EIA-1608-08_AVX-J"
 			(at 93.6752 31.75 0)
 			(effects
@@
 			)
 		)
-		(property "Footprint" ""
+		(property "Footprint" "Button_Switch_SMD:Nidec_Copal_CAS-120A"
 			(at 21.59 124.46 0)
 			(effects
@@
 			)
 		)
-		(property "Footprint" ""
+		(property "Footprint" "Capacitor_Tantalum_SMD:CP_EIA-1608-08_AVX-J"
 			(at 60.6552 46.99 0)
 			(effects
@@
 			)
 		)
-		(property "Footprint" ""
+		(property "Footprint" "Capacitor_Tantalum_SMD:CP_EIA-1608-08_AVX-J"
 			(at 181.3052 78.74 0)
 			(effects
@@
 			)
 		)
-		(property "Footprint" ""
+		(property "Footprint" "Capacitor_Tantalum_SMD:CP_EIA-1608-08_AVX-J"
 			(at 65.7352 173.99 0)
 			(effects
@@
 			)
 		)
-		(property "Footprint" ""
+		(property "Footprint" "Connector:BJB_Pico_46.110.1001_Receptacle_Horizontal"
 			(at 200.66 30.48 0)
 			(effects
@@
 			)
 		)
-		(property "Footprint" ""
+		(property "Footprint" "Capacitor_Tantalum_SMD:CP_EIA-1608-10_AVX-L"
 			(at 41.6052 173.99 0)
 			(effects
@@
 			)
 		)
-		(property "Footprint" ""
+		(property "Footprint" "Resistor_SMD:R_0201_0603Metric"
 			(at 31.242 115.57 90)
 			(effects
@@
 			)
 		)
-		(property "Footprint" ""
+		(property "Footprint" "Resistor_SMD:R_0201_0603Metric"
 			(at 225.552 60.96 90)
 			(effects
@@
 			)
 		)
-		(property "Footprint" ""
+		(property "Footprint" "Resistor_SMD:R_0201_0603Metric"
 			(at 267.97 24.892 90)
 			(effects
@@
 			)
 		)
-		(property "Footprint" ""
+		(property "Footprint" "Capacitor_Tantalum_SMD:CP_EIA-1608-08_AVX-J"
 			(at 47.9552 46.99 0)
 			(effects
@@
 			)
 		)
-		(property "Footprint" ""
+		(property "Footprint" "Capacitor_Tantalum_SMD:CP_EIA-1608-08_AVX-J"
 			(at 101.2952 31.75 0)
 			(effects
@@
 			)
 		)
-		(property "Footprint" ""
+		(property "Footprint" "Button_Switch_SMD:Nidec_Copal_CAS-120A"
 			(at 254 76.2 0)
 			(effects
@@
 			)
 		)
-		(property "Footprint" ""
+		(property "Footprint" "Capacitor_Tantalum_SMD:CP_EIA-1608-08_AVX-J"
 			(at 33.9852 127 0)
 			(effects
@@
 			)
 		)
-		(property "Footprint" ""
+		(property "Footprint" "Capacitor_Tantalum_SMD:CP_EIA-1608-08_AVX-J"
 			(at 53.0352 173.99 0)
 			(effects
@@
 			)
 		)
-		(property "Footprint" ""
+		(property "Footprint" "Capacitor_Tantalum_SMD:CP_EIA-1608-08_AVX-J"
 			(at 88.5952 173.99 0)
 			(effects
@@
 			)
 		)
-		(property "Footprint" ""
+		(property "Footprint" "Capacitor_Tantalum_SMD:CP_EIA-1608-08_AVX-J"
 			(at 261.3152 34.29 0)
 			(effects
@@
 			)
 		)
-		(property "Footprint" ""
+		(property "Footprint" "Resistor_SMD:R_0201_0603Metric"
 			(at 234.95 70.358 90)
 			(effects
@@
 			)
 		)
-		(property "Footprint" ""
+		(property "Footprint" "Capacitor_Tantalum_SMD:CP_EIA-1608-08_AVX-J"
 			(at 242.2652 34.29 0)
 			(effects
@@
 			)
 		)
-		(property "Footprint" ""
+		(property "Footprint" "Capacitor_Tantalum_SMD:CP_EIA-1608-08_AVX-J"
 			(at 100.0252 173.99 0)
 			(effects

Commit message: update
Connections:
- net FLASH_CS is gone; now on net ~{FLASH_CS}: U1.56 (QSPI_SS)
- net FLASH_D2 is gone; now on net ~{FLASH_D2}: U1.54 (QSPI_SD2)
- net I2CO_SCL is gone; now on net I2C0_SCL: U1.3 (GPIO1)
- net ~{FLASH_CS}: now reaches R5.2, R6.1, U2.1 (~{CS})
- net 12CO_SCL renamed I2C0_SCL
- net I2CO_SDA renamed I2C0_SDA
Other:
- note removed: "I2CO_SCL"
- note removed: "I2CO_SDA"
- note removed: "~{FLASH_CS}"
Changed lines of the file:
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@@
 		)
 	)
-	(text "I2CO_SDA"
-		(exclude_from_sim no)
-		(at 118.364 52.578 0)
-		(effects
-			(font
-				(size 1.27 1.27)
-			)
-		)
-	)
-	(text "I2CO_SCL"
-		(exclude_from_sim no)
-		(at 118.364 55.118 0)
-		(effects
-			(font
-				(size 1.27 1.27)
-			)
-		)
-	)
-	(text "~{FLASH_CS}"
-		(exclude_from_sim no)
-		(at 216.916 67.818 0)
-		(effects
-			(font
-				(size 1.27 1.27)
-			)
-		)
-	)
 	(junction
 		(at 185.42 81.28)
@@
 	)
 	(junction
-		(at 60.96 33.02)
-		(diameter 0)
-		(color 0 0 0 0)
-	)
-	(junction
 		(at 52.07 163.83)
 		(diameter 0)
@@
 	)
 	(junction
+		(at 57.15 33.02)
+		(diameter 0)
+		(color 0 0 0 0)
+	)
+	(junction
 		(at 53.34 35.56)
 		(diameter 0)
@@
 	(wire
 		(pts
-			(xy 60.96 33.02) (xy 69.85 33.02)
+			(xy 57.15 33.02) (xy 69.85 33.02)
 		)
 		(stroke
@@
 	(wire
 		(pts
-			(xy 53.34 33.02) (xy 60.96 33.02)
+			(xy 53.34 33.02) (xy 57.15 33.02)
 		)
 		(stroke
@@
 		)
 	)
-	(label "FLASH_D2"
+	(label "~{FLASH_D2}"
 		(at 52.07 78.74 0)
 		(effects
@@
 		)
 	)
-	(label "I2CO_SDA"
+	(label "I2C0_SDA"
 		(at 181.61 31.75 180)
 		(effects
@@
 		)
 	)
+	(label "~{FLASH_CS}"
+		(at 213.36 68.58 0)
+		(effects
+			(font
+				(size 1.27 1.27)
+			)
+			(justify left bottom)
+		)
+	)
 	(label "XOUT"
 		(at 52.07 101.6 0)
@@
 		)
 	)
-	(label "FLASH_CS"
+	(label "~{FLASH_CS}"
 		(at 52.07 68.58 0)
 		(effects
@@
 		)
 	)
+	(label "I2C0_SCL"
+		(at 114.3 55.88 0)
+		(effects
+			(font
+				(size 1.27 1.27)
+			)
+			(justify left bottom)
+		)
+	)
 	(label "SWCLK"
 		(at 214.63 27.94 180)
@@
 		)
 	)
+	(label "I2C0_SDA"
+		(at 114.3 53.34 0)
+		(effects
+			(font
+				(size 1.27 1.27)
+			)
+			(justify left bottom)
+		)
+	)
 	(label "XIN"
 		(at 52.07 99.06 0)
@@
 		)
 	)
-	(label "12CO_SCL"
+	(label "I2C0_SCL"
 		(at 181.61 29.21 180)
 		(effects
@@
 		)
 	)
-	(hierarchical_label "I2CO_SDA"
+	(hierarchical_label "I2C0_SDA"
 		(shape output)
 		(at 127 53.34 0)
@@
 		)
 	)
-	(hierarchical_label "I2CO_SCL"
+	(hierarchical_label "I2C0_SCL"
 		(shape output)
 		(at 127 55.88 0)
@@
 	)
 	(symbol
-		(lib_id "power:GND")
-		(at 53.34 53.34 0)
-		(unit 1)
-		(exclude_from_sim no)
-		(in_bom yes)
-		(on_board yes)
-		(dnp no)
-		(fields_autoplaced yes)
-		(property "Reference" "#PWR067"
-			(at 53.34 59.69 0)
-			(effects
-				(font
-					(size 1.27 1.27)
-				)
-				(hide yes)
-			)
-		)
-		(property "Value" "GND"
-			(at 53.34 58.42 0)
-			(effects
-				(font
-					(size 1.27 1.27)
-				)
-			)
-		)
-		(property "Footprint" ""
-			(at 53.34 53.34 0)
-			(effects
-				(font
-					(size 1.27 1.27)
-				)
-				(hide yes)
-			)
-		)
-		(property "Datasheet" ""
-			(at 53.34 53.34 0)
-			(effects
-				(font
-					(size 1.27 1.27)
-				)
-				(hide yes)
-			)
-		)
-		(property "Description" "Power symbol creates a global label with name \"GND\" , ground"
-			(at 53.34 53.34 0)
-			(effects
-				(font
-					(size 1.27 1.27)
-				)
-				(hide yes)
-			)
-		)
-		(pin "1"
-		)
-		(instances
-			(project ""
-				(path "/13844229-b559-4868-a710-53f590233cb2/995b0e09-2caa-42c1-89e8-61a13534fe57"
-					(reference "#PWR067")
-					(unit 1)
-				)
-			)
-		)
-	)
-	(symbol
 		(lib_id "power:+1V1")
 		(at 97.79 21.59 0)
@@
 	)
 	(symbol
-		(lib_id "power:PWR_FLAG")
-		(at 60.96 33.02 0)
-		(unit 1)
-		(exclude_from_sim no)
-		(in_bom yes)
-		(on_board yes)
-		(dnp no)
-		(fields_autoplaced yes)
-		(property "Reference" "#FLG03"
-			(at 60.96 31.115 0)
-			(effects
-				(font
-					(size 1.27 1.27)
-				)
-				(hide yes)
-			)
-		)
-		(property "Value" "PWR_FLAG"
-			(at 60.96 27.94 0)
-			(effects
-				(font
-					(size 1.27 1.27)
-				)
-			)
-		)
-		(property "Footprint" ""
-			(at 60.96 33.02 0)
-			(effects
-				(font
-					(size 1.27 1.27)
-				)
-				(hide yes)
-			)
-		)
-		(property "Datasheet" "~"
-			(at 60.96 33.02 0)
-			(effects
-				(font
-					(size 1.27 1.27)
-				)
-				(hide yes)
-			)
-		)
-		(property "Description" "Special symbol for telling ERC where power comes from"
-			(at 60.96 33.02 0)
-			(effects
-				(font
-					(size 1.27 1.27)
-				)
-				(hide yes)
-			)
-		)
-		(pin "1"
-		)
-		(instances
-			(project ""
-				(path "/13844229-b559-4868-a710-53f590233cb2/995b0e09-2caa-42c1-89e8-61a13534fe57"
-					(reference "#FLG03")
-					(unit 1)
-				)
-			)
-		)
-	)
-	(symbol
 		(lib_id "Device:C")
 		(at 92.71 27.94 0)
@@
 	)
 	(symbol
+		(lib_id "power:PWR_FLAG")
+		(at 57.15 33.02 0)
+		(unit 1)
+		(exclude_from_sim no)
+		(in_bom yes)
+		(on_board yes)
+		(dnp no)
+		(fields_autoplaced yes)
+		(property "Reference" "#FLG01"
+			(at 57.15 31.115 0)
+			(effects
+				(font
+					(size 1.27 1.27)
+				)
+				(hide yes)
+			)
+		)
+		(property "Value" "PWR_FLAG"
+			(at 57.15 27.94 0)
+			(effects
+				(font
+					(size 1.27 1.27)
+				)
+			)
+		)
+		(property "Footprint" ""
+			(at 57.15 33.02 0)
+			(effects
+				(font
+					(size 1.27 1.27)
+				)
+				(hide yes)
+			)
+		)
+		(property "Datasheet" "~"
+			(at 57.15 33.02 0)
+			(effects
+				(font
+					(size 1.27 1.27)
+				)
+				(hide yes)
+			)
+		)
+		(property "Description" "Special symbol for telling ERC where power comes from"
+			(at 57.15 33.02 0)
+			(effects
+				(font
+					(size 1.27 1.27)
+				)
+				(hide yes)
+			)
+		)
+		(pin "1"
+		)
+		(instances
+			(project ""
+				(path "/13844229-b559-4868-a710-53f590233cb2/995b0e09-2caa-42c1-89e8-61a13534fe57"
+					(reference "#FLG01")
+					(unit 1)
+				)
+			)
+		)
+	)
+	(symbol
 		(lib_id "Device:R")
 		(at 267.97 26.67 270)
@@
 					(unit 1)
 				)
+			)
+		)
+	)
+	(symbol
+		(lib_id "power:GND")
+		(at 53.34 53.34 0)
+		(unit 1)
+		(exclude_from_sim no)
+		(in_bom yes)
+		(on_board yes)
+		(dnp no)
+		(fields_autoplaced yes)
+		(property "Reference" "#PWR067"
+			(at 53.34 59.69 0)
+			(effects
+				(font
+					(size 1.27 1.27)
+				)
+				(hide yes)
+			)
+		)
+		(property "Value" "GND"
+			(at 53.34 58.42 0)
+			(effects
+				(font
+					(size 1.27 1.27)
+				)
+			)
+		)
+		(property "Footprint" ""
+			(at 53.34 53.34 0)
+			(effects
+				(font
+					(size 1.27 1.27)
+				)
+				(hide yes)
+			)
+		)
+		(property "Datasheet" ""
+			(at 53.34 53.34 0)
+			(effects
+				(font
+					(size 1.27 1.27)
+				)
+				(hide yes)
+			)
+		)
+		(property "Description" "Power symbol creates a global label with name \"GND\" , ground"
+			(at 53.34 53.34 0)
+			(effects
+				(font
+					(size 1.27 1.27)
+				)
+				(hide yes)
+			)
+		)
+		(pin "1"
+		)
+		(instances
+			(project ""
+				(path "/13844229-b559-4868-a710-53f590233cb2/995b0e09-2caa-42c1-89e8-61a13534fe57"
+					(reference "#PWR067")
+					(unit 1)
+				)

Commit message: update
Changed lines of the file:
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@@
 	)
 	(junction
+		(at 59.69 33.02)
+		(diameter 0)
+		(color 0 0 0 0)
+	)
+	(junction
 		(at 241.3 26.67)
 		(diameter 0)
@@
 	)
 	(junction
-		(at 57.15 33.02)
-		(diameter 0)
-		(color 0 0 0 0)
-	)
-	(junction
 		(at 53.34 35.56)
 		(diameter 0)
@@
 	(wire
 		(pts
+			(xy 59.69 29.21) (xy 59.69 33.02)
+		)
+		(stroke
+			(width 0)
+			(type default)
+		)
+	)
+	(wire
+		(pts
 			(xy 241.3 38.1) (xy 251.46 38.1)
 		)
@@
 	(wire
 		(pts
+			(xy 59.69 33.02) (xy 69.85 33.02)
+		)
+		(stroke
+			(width 0)
+			(type default)
+		)
+	)
+	(wire
+		(pts
 			(xy 33.02 129.54) (xy 26.67 129.54)
 		)
@@
 	(wire
 		(pts
-			(xy 57.15 33.02) (xy 69.85 33.02)
-		)
-		(stroke
-			(width 0)
-			(type default)
-		)
-	)
-	(wire
-		(pts
 			(xy 248.92 68.58) (xy 248.92 71.12)
 		)
@@
 	(wire
 		(pts
-			(xy 53.34 33.02) (xy 57.15 33.02)
+			(xy 53.34 33.02) (xy 59.69 33.02)
 		)
 		(stroke
@@
 	)
 	(symbol
+		(lib_name "+1V1_1")
 		(lib_id "power:+1V1")
 		(at 69.85 33.02 0)
@@
 	(symbol
 		(lib_id "power:PWR_FLAG")
-		(at 57.15 33.02 0)
+		(at 59.69 29.21 0)
 		(unit 1)
 		(exclude_from_sim no)
@@
 		(on_board yes)
 		(dnp no)
-		(fields_autoplaced yes)
 		(property "Reference" "#FLG01"
-			(at 57.15 31.115 0)
+			(at 59.69 27.305 0)
 			(effects
 				(font
@@
 		)
 		(property "Value" "PWR_FLAG"
-			(at 57.15 27.94 0)
+			(at 59.944 24.13 0)
 			(effects
 				(font
@@
 		)
 		(property "Footprint" ""
-			(at 57.15 33.02 0)
+			(at 59.69 29.21 0)
 			(effects
 				(font
@@
 		)
 		(property "Datasheet" "~"
-			(at 57.15 33.02 0)
+			(at 59.69 29.21 0)
 			(effects
 				(font
@@
 		)
 		(property "Description" "Special symbol for telling ERC where power comes from"
-			(at 57.15 33.02 0)
+			(at 59.69 29.21 0)
 			(effects
 				(font

Commit message: update
Parts:
- C10, C11, C12, C13, C14, C15, C16, C17, C18, C19, C20, C21, C22, C23: footprint Capacitor_Tantalum_SMD:CP_EIA-1608-08_AVX-J -> Capacitor_SMD:C_0603_1608Metric
- C9: footprint Capacitor_Tantalum_SMD:CP_EIA-1608-10_AVX-L -> Capacitor_SMD:C_0603_1608Metric
- J2: footprint Connector:BJB_Pico_46.110.1001_Receptacle_Horizontal -> Connector_PinHeader_2.54mm:PinHeader_1x03_P2.54mm_Vertical
- R4, R5, R6: footprint Resistor_SMD:R_0201_0603Metric -> Resistor_SMD:R_0603_1608Metric
- R7: value R -> 1k; footprint Resistor_SMD:R_0201_0603Metric -> Resistor_SMD:R_0603_1608Metric
- SW1, SW2: footprint Button_Switch_SMD:Nidec_Copal_CAS-120A -> Button_Switch_SMD:SW_SPST_EVQP0
Changed lines of the file:
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@@
 		(stroke
 			(width 0)
-			(type default)
+			(type dash)
 		)
 		(fill
@@
 		(stroke
 			(width 0)
-			(type default)
+			(type dash)
 		)
 		(fill
@@
 		(stroke
 			(width 0)
-			(type default)
+			(type dash)
 		)
 		(fill
@@
 		(stroke
 			(width 0)
-			(type default)
+			(type dash)
 		)
 		(fill
@@
 		(stroke
 			(width 0)
-			(type default)
+			(type dash)
 		)
 		(fill
@@
 			)
 		)
-		(property "Footprint" "Capacitor_Tantalum_SMD:CP_EIA-1608-08_AVX-J"
+		(property "Footprint" "Capacitor_SMD:C_0603_1608Metric"
 			(at 77.1652 173.99 0)
 			(effects
@@
 			)
 		)
-		(property "Footprint" "Capacitor_Tantalum_SMD:CP_EIA-1608-08_AVX-J"
+		(property "Footprint" "Capacitor_SMD:C_0603_1608Metric"
 			(at 112.7252 173.99 0)
 			(effects
@@
 			)
 		)
-		(property "Footprint" "Capacitor_Tantalum_SMD:CP_EIA-1608-08_AVX-J"
+		(property "Footprint" "Capacitor_SMD:C_0603_1608Metric"
 			(at 93.6752 31.75 0)
 			(effects
@@
 			)
 		)
-		(property "Footprint" "Button_Switch_SMD:Nidec_Copal_CAS-120A"
+		(property "Footprint" "Button_Switch_SMD:SW_SPST_EVQP0"
 			(at 21.59 124.46 0)
 			(effects
@@
 			)
 		)
-		(property "Footprint" "Capacitor_Tantalum_SMD:CP_EIA-1608-08_AVX-J"
+		(property "Footprint" "Capacitor_SMD:C_0603_1608Metric"
 			(at 60.6552 46.99 0)
 			(effects
@@
 			)
 		)
-		(property "Footprint" "Capacitor_Tantalum_SMD:CP_EIA-1608-08_AVX-J"
+		(property "Footprint" "Capacitor_SMD:C_0603_1608Metric"
 			(at 181.3052 78.74 0)
 			(effects
@@
 			)
 		)
-		(property "Footprint" "Capacitor_Tantalum_SMD:CP_EIA-1608-08_AVX-J"
+		(property "Footprint" "Capacitor_SMD:C_0603_1608Metric"
 			(at 65.7352 173.99 0)
 			(effects
@@
 			)
 		)
-		(property "Footprint" "Connector:BJB_Pico_46.110.1001_Receptacle_Horizontal"
+		(property "Footprint" "Connector_PinHeader_2.54mm:PinHeader_1x03_P2.54mm_Vertical"
 			(at 200.66 30.48 0)
 			(effects
@@
 			)
 		)
-		(property "Footprint" "Capacitor_Tantalum_SMD:CP_EIA-1608-10_AVX-L"
+		(property "Footprint" "Capacitor_SMD:C_0603_1608Metric"
 			(at 41.6052 173.99 0)
 			(effects
@@
 			)
 		)
-		(property "Footprint" "Resistor_SMD:R_0201_0603Metric"
+		(property "Footprint" "Resistor_SMD:R_0603_1608Metric"
 			(at 31.242 115.57 90)
 			(effects
@@
 			)
 		)
-		(property "Footprint" "Resistor_SMD:R_0201_0603Metric"
+		(property "Footprint" "Resistor_SMD:R_0603_1608Metric"
 			(at 225.552 60.96 90)
 			(effects
@@
 			)
 		)
-		(property "Value" "R"
+		(property "Value" "1k"
 			(at 267.97 22.86 90)
 			(effects
@@
 			)
 		)
-		(property "Footprint" "Resistor_SMD:R_0201_0603Metric"
+		(property "Footprint" "Resistor_SMD:R_0603_1608Metric"
 			(at 267.97 24.892 90)
 			(effects
@@
 			)
 		)
-		(property "Footprint" "Capacitor_Tantalum_SMD:CP_EIA-1608-08_AVX-J"
+		(property "Footprint" "Capacitor_SMD:C_0603_1608Metric"
 			(at 47.9552 46.99 0)
 			(effects
@@
 			)
 		)
-		(property "Footprint" "Capacitor_Tantalum_SMD:CP_EIA-1608-08_AVX-J"
+		(property "Footprint" "Capacitor_SMD:C_0603_1608Metric"
 			(at 101.2952 31.75 0)
 			(effects
@@
 			)
 		)
-		(property "Footprint" "Button_Switch_SMD:Nidec_Copal_CAS-120A"
+		(property "Footprint" "Button_Switch_SMD:SW_SPST_EVQP0"
 			(at 254 76.2 0)
 			(effects
@@
 			)
 		)
-		(property "Footprint" "Capacitor_Tantalum_SMD:CP_EIA-1608-08_AVX-J"
+		(property "Footprint" "Capacitor_SMD:C_0603_1608Metric"
 			(at 33.9852 127 0)
 			(effects
@@
 			)
 		)
-		(property "Footprint" "Capacitor_Tantalum_SMD:CP_EIA-1608-08_AVX-J"
+		(property "Footprint" "Capacitor_SMD:C_0603_1608Metric"
 			(at 53.0352 173.99 0)
 			(effects
@@
 			)
 		)
-		(property "Footprint" "Capacitor_Tantalum_SMD:CP_EIA-1608-08_AVX-J"
+		(property "Footprint" "Capacitor_SMD:C_0603_1608Metric"
 			(at 88.5952 173.99 0)
 			(effects
@@
 			)
 		)
-		(property "Footprint" "Capacitor_Tantalum_SMD:CP_EIA-1608-08_AVX-J"
+		(property "Footprint" "Capacitor_SMD:C_0603_1608Metric"
 			(at 261.3152 34.29 0)
 			(effects
@@
 			)
 		)
-		(property "Footprint" "Resistor_SMD:R_0201_0603Metric"
+		(property "Footprint" "Resistor_SMD:R_0603_1608Metric"
 			(at 234.95 70.358 90)
 			(effects
@@
 			)
 		)
-		(property "Footprint" "Capacitor_Tantalum_SMD:CP_EIA-1608-08_AVX-J"
+		(property "Footprint" "Capacitor_SMD:C_0603_1608Metric"
 			(at 242.2652 34.29 0)
 			(effects
@@
 			)
 		)
-		(property "Footprint" "Capacitor_Tantalum_SMD:CP_EIA-1608-08_AVX-J"
+		(property "Footprint" "Capacitor_SMD:C_0603_1608Metric"
 			(at 100.0252 173.99 0)
 			(effects
