File: hard/mcu.kicad_sch (KiCad schematic)
At the start: 26 parts, among them J2 Conn_01x03, SW1 RESET_SW, SW2 PROG_SW, U1 RP2040, U2 W25Q128JVE, U3 AT24C256, Y1 12MHz

Commit message: update
Parts:
- removed U1: RP2040, Package_DFN_QFN:QFN-56-1EP_7x7mm_P0.4mm_EP3.2x3.2mm, symbol MCU_RaspberryPi:RP2040
- removed U2: W25Q128JVE, Package_SON:WSON-8-1EP_8x6mm_P1.27mm_EP3.4x4.3mm, symbol Memory_Flash:W25Q128JVE
- removed U3: AT24C256, Package_SO:SOIC-8_3.9x4.9mm_P1.27mm, symbol Memory_EEPROM:AT24CS01-SSHM
- removed Y1: 12MHz, Crystal:Crystal_SMD_3225-4Pin_3.2x2.5mm_HandSoldering, symbol Device:Crystal_GND23
- added U1: RP2040, Package_DFN_QFN:QFN-56-1EP_7x7mm_P0.4mm_EP3.2x3.2mm, symbol libs:RP2040
- added U2: W25Q16JVUSSQ, Package_SON:WSON-8-1EP_8x6mm_P1.27mm_EP3.4x4.3mm, symbol libs:W25Q128JVE
- added U3: AT24C256, Package_SO:SOIC-8_3.9x4.9mm_P1.27mm, symbol libs:AT24CS01-SSHM
- added Y1: 12MHz, Crystal:Crystal_SMD_3225-4Pin_3.2x2.5mm_HandSoldering, symbol libs:Crystal_GND23
Connections:
- net +1V1: now also U1.23 (DVDD), U1.45 (VREG_VOUT), U1.50 (DVDD)
- net +3.3VA: now also U1.43 (ADC_AVDD)
- net +3V3: now also U1.1 (IOVDD), U1.10 (IOVDD), U1.22 (IOVDD), U1.33 (IOVDD), U1.42 (IOVDD), U1.44 (VREG_IN), U1.48 (USB_VDD), U1.49 (IOVDD), U2.8 (VCC), U3.8 (VCC)
- net 5V_EN: now also U1.14 (GPIO11)
- net BUZZER_PWM: now also U1.32 (GPIO21)
- net C_XOUT: now also Y1.4
- net ESP-01_EN: now also U1.5 (GPIO3)
- net FLASH_CLK: now also U1.52 (QSPI_SCLK), U2.6 (CLK)
- net FLASH_D0: now also U1.53 (QSPI_SD0), U2.5 (DI_IOO)
- net FLASH_D1: now also U1.55 (QSPI_SD1), U2.2 (DO_IO1)
- net FLASH_D3: now also U1.51 (QSPI_SD3), U2.7 (HOLD_IO3)
- net GND: now also U1.19 (TESTEN), U1.57 (GND), U2.4 (GND), U3.1 (A0), U3.2 (A1), U3.4 (GND), U3.7 (WP), Y1.2, Y1.3
- net GPS_EN: now also U1.29 (GPIO18)
- net GPS_PPS: now also U1.30 (GPIO19)
- net GPS_RST: now also U1.15 (GPIO12)
- net I2C0_SCL: now also U1.3 (GPIO1), U3.6 (SCL)
- net I2C0_SDA: now also U1.2 (GPIO0), U3.5 (SDA)
- net INT1_ACC: now also U1.17 (GPIO14)
- net INT2_ACC: now also U1.18 (GPIO15)
- net LED_ALIVE: now also U1.31 (GPIO20)
- net OUTPUT_USBEN: now also U1.39 (GPIO27/ADC1)
- net PWM_SERVO1: now also U1.11 (GPIO8)
- net PWM_SERVO2: now also U1.12 (GPIO9)
- net PWM_SERVO3: now also U1.9 (GPIO7)
- net RGB_LED: now also U1.16 (GPIO13)
- net SWCLK: now also U1.24 (SWCLK)
- net SWDIO: now also U1.25 (SWD)
- net SW_DOWN: now also U1.35 (GPIO23)
- net SW_LEFT: now also U1.37 (GPIO25)
- net SW_RIGHT: now also U1.36 (GPIO24)
- net SW_UP: now also U1.34 (GPIO22)
- net TEMP_SENS: now also U1.38 (GPIO26/ADC0)
- net UART0_RX: now also U1.28 (GPIO17)
- net UART0_TX: now also U1.27 (GPIO16)
- net UART1_RX: now also U1.7 (GPIO5)
- net UART1_TX: now also U1.6 (GPIO4)
- net USB_DN: now also U1.46 (USB_DM)
- net USB_DP: now also U1.47 (USB_DP)
- net USB_ID: now also U1.4 (GPIO2)
- net VBAT: now also U1.40 (GPIO28/ADC2)
- net XIN: now also U1.20 (XIN), Y1.1
- net XOUT: now also U1.21 (XOUT)
- net ~{FLASH_CS}: now also U1.56 (QSPI_SS), U2.1 (~{CS})
- net ~{FLASH_D2}: now also U1.54 (QSPI_SD2), U2.3 (WP_IO2)
- net at C11.1, R4.2, SW1.2: now also U1.26 (RUN)

Commit message: update
Parts:
- U2: footprint Package_SON:WSON-8-1EP_8x6mm_P1.27mm_EP3.4x4.3mm -> Package_SO:SOIC-8_5.3x5.3mm_P1.27mm
Connections:
- net ~{USB_BOOT}: now reaches R6.2, SW2.1 (A), SW2.2 (A)
Other:
- note removed: "~{USB_BOOT}"
- title: (none) -> Microcontrollore e Memorie
- moved on the sheet: C10, C12, C13, C15, C17, C18, C9
