File: hard/mcu.kicad_sch (KiCad schematic)
At the start: 26 parts, among them J2 Conn_01x03, SW1 RESET_SW, SW2 PROG_SW, U1 RP2040, U2 W25Q16JVUSSQ, U3 AT24C256, Y1 12MHz

Commit message: update
Parts:
- SW2: symbol Switch:SW_MEC_5G -> Switch:SW_Push
Connections:
- net GND: now also SW2.2; no longer SW2.3 (B), SW2.4 (B)
- net ~{USB_BOOT}: no longer SW2.2 (A)
Changed lines of the file:
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@@
 	)
 	(symbol
-		(lib_id "Switch:SW_MEC_5G")
+		(lib_id "Switch:SW_Push")
 		(at 248.92 76.2 270)
 		(unit 1)
@@
 			)
 		)
-		(property "Datasheet" "http://www.apem.com/int/index.php?controller=attachment&id_attachment=488"
+		(property "Datasheet" "~"
 			(at 254 76.2 0)
 			(effects
@@
 			)
 		)
-		(property "Description" "MEC 5G single pole normally-open tactile switch"
+		(property "Description" "Push button switch, generic, two pins"
 			(at 248.92 76.2 0)
 			(effects
@@
 		(pin "1"
 		)
-		(pin "3"
-		)
 		(pin "2"
 		)
-		(pin "4"
-		)
 		(instances
