File: hard/ui.kicad_sch (KiCad schematic)
At the start: 0 parts

Commit message: update
Parts:
- added BZ2: Buzzer, symbol Device:Buzzer
- added C10, C11, C12, C13: C, symbol Device:C
- added C27: 4.7u, symbol Device:C
- added C28: 100n, symbol Device:C
- added D18: D, symbol Device:D
- added D19: LED, symbol Device:LED
- added Q3: DTD123Y, symbol Transistor_BJT:DTD123Y
- added R10, R11, R14, R15, R20: R, symbol Device:R
- added SW10, SW7, SW8, SW9: SW_MEC_5G, symbol Switch:SW_MEC_5G
Connections:
- new net: D19.2 (A), R20.2
- new net: BZ2.2 (-), D18.2 (A), Q3.3 (C)
- new net +3V3: C27.1, C28.1
- new net BUZZER: Q3.1 (B)
- new net GND: C10.2, C11.2, C12.2, C13.2, C27.2, C28.2, D19.1 (K), Q3.2 (E), SW10.3 (B), SW10.4 (B), SW7.3 (B), SW7.4 (B), SW8.3 (B), SW8.4 (B), SW9.3 (B), SW9.4 (B)
- new net LED_ALIVE: R20.1
- new net SW_DOWN: C10.1, C11.1, C12.1, C13.1, R10.2, R11.2, R14.2, R15.2, SW10.1 (A), SW10.2 (A), SW7.1 (A), SW7.2 (A), SW8.1 (A), SW8.2 (A), SW9.1 (A), SW9.2 (A)
- new net VDD: BZ2.1 (+), D18.1 (K), R10.1, R11.1, R14.1, R15.1
Other:
- removed sheet buzzer
- removed sheet display
- removed sheet display_buttons
- removed sheet led_alive

Commit message: update
Parts:
- added U4: oled_0.96"_128x64px, Display:EA_DOGS104X-A, symbol Display_Graphic:EA_DOGS104B-A
- C24: renamed from C10; value C -> 100n
- C25: renamed from C11; value C -> 100n
- C26: renamed from C13; value C -> 100n
- C27: renamed from C12; value C -> 100n
- D10: renamed from D19; value LED -> LED_alive
- D9: renamed from D18; value D -> 1N4148
- Q2: renamed from Q3; value DTD123Y -> PDTC114YT
- R11: renamed from R14; value R -> 470k
- R12: renamed from R20; value R -> 470
- R8: renamed from R10; value R -> 470k
- R9: renamed from R11; value R -> 470k
- SW3: renamed from SW7; value SW_MEC_5G -> SW_U
- SW4: renamed from SW8; value SW_MEC_5G -> SW_L
- SW5: renamed from SW10; value SW_MEC_5G -> SW_R
- SW6: renamed from SW9; value SW_MEC_5G -> SW_D
- renumbered BZ2 to BZ1, C27 to C28, C28 to C29, R15 to R10
Connections:
- net +3V3: now also R10.1, R11.1, R8.1, R9.1, U4.2 (VDD)
- net GND: now also U4.1 (GND)
- net SCL_DISPLAY: now also U4.3 (SCK)
- net SDA_DISPLAY: now also U4.4 (SDA)
- net SW_DOWN: no longer C24.1, C25.1, C26.1, R10.2, R8.2, R9.2, SW3.1 (A), SW3.2 (A), SW4.1 (A), SW4.2 (A), SW5.1 (A), SW5.2 (A)
- net VDD: no longer R10.1, R11.1, R8.1, R9.1
- new net SW_LEFT: C25.1, R9.2, SW4.1 (A), SW4.2 (A)
- new net SW_RIGHT: C26.1, R10.2, SW5.1 (A), SW5.2 (A)
- new net SW_UP: C24.1, R8.2, SW3.1 (A), SW3.2 (A)
Other:
- note added: "Buzzer"
- note added: "Display"
- note added: "LED alive"
- note added: "Pulsanti Display"
- moved on the sheet: BZ1, C24, C25, C26, C27, C28, C29, D10, D9, Q2, R10, R11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

Commit message: update
Parts:
- BZ1: footprint (none) -> Buzzer_Beeper:Buzzer_12x9.5RM7.6
- C24, C25, C26, C27, C28, C29: footprint (none) -> Capacitor_Tantalum_SMD:CP_EIA-1608-08_AVX-J
- D10: footprint (none) -> LED_SMD:LED_0805_2012Metric
- D9: footprint (none) -> Diode_SMD:D_SOD-123
- Q2: footprint (none) -> Package_TO_SOT_SMD:SOT-23
- R10, R11, R12, R8, R9: footprint (none) -> Resistor_SMD:R_0201_0603Metric
- SW3, SW4, SW5, SW6: footprint (none) -> Button_Switch_SMD:Nidec_Copal_CAS-120A
Changed lines of the file:
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@@
 			)
 		)
-		(property "Footprint" ""
+		(property "Footprint" "LED_SMD:LED_0805_2012Metric"
 			(at 135.89 86.36 0)
 			(effects
@@
 			)
 		)
-		(property "Footprint" ""
+		(property "Footprint" "Resistor_SMD:R_0201_0603Metric"
 			(at 87.122 26.67 90)
 			(effects
@@
 			)
 		)
-		(property "Footprint" ""
+		(property "Footprint" "Button_Switch_SMD:Nidec_Copal_CAS-120A"
 			(at 58.42 87.63 0)
 			(effects
@@
 			)
 		)
-		(property "Footprint" ""
+		(property "Footprint" "Button_Switch_SMD:Nidec_Copal_CAS-120A"
 			(at 106.68 87.63 0)
 			(effects
@@
 			)
 		)
-		(property "Footprint" ""
+		(property "Footprint" "Diode_SMD:D_SOD-123"
 			(at 137.16 31.75 0)
 			(effects
@@
 			)
 		)
-		(property "Footprint" ""
+		(property "Footprint" "Capacitor_Tantalum_SMD:CP_EIA-1608-08_AVX-J"
 			(at 89.8652 93.98 0)
 			(effects
@@
 			)
 		)
-		(property "Footprint" ""
+		(property "Footprint" "Resistor_SMD:R_0201_0603Metric"
 			(at 87.122 73.66 90)
 			(effects
@@
 			)
 		)
-		(property "Footprint" ""
+		(property "Footprint" "Buzzer_Beeper:Buzzer_12x9.5RM7.6"
 			(at 151.765 30.48 90)
 			(effects
@@
 			)
 		)
-		(property "Footprint" ""
+		(property "Footprint" "Resistor_SMD:R_0201_0603Metric"
 			(at 38.862 73.66 90)
 			(effects
@@
 			)
 		)
-		(property "Footprint" ""
+		(property "Footprint" "Capacitor_Tantalum_SMD:CP_EIA-1608-08_AVX-J"
 			(at 41.6052 93.98 0)
 			(effects
@@
 			)
 		)
-		(property "Footprint" ""
+		(property "Footprint" "Button_Switch_SMD:Nidec_Copal_CAS-120A"
 			(at 53.34 41.91 0)
 			(effects
@@
 			)
 		)
-		(property "Footprint" ""
+		(property "Footprint" "Capacitor_Tantalum_SMD:CP_EIA-1608-08_AVX-J"
 			(at 195.2752 45.72 0)
 			(effects
@@
 			)
 		)
-		(property "Footprint" ""
+		(property "Footprint" "Resistor_SMD:R_0201_0603Metric"
 			(at 134.112 78.74 90)
 			(effects
@@
 			)
 		)
-		(property "Footprint" ""
+		(property "Footprint" "Capacitor_Tantalum_SMD:CP_EIA-1608-08_AVX-J"
 			(at 89.8652 46.99 0)
 			(effects
@@
 			)
 		)
-		(property "Footprint" ""
+		(property "Footprint" "Button_Switch_SMD:Nidec_Copal_CAS-120A"
 			(at 101.6 41.91 0)
 			(effects
@@
 			)
 		)
-		(property "Footprint" ""
+		(property "Footprint" "Resistor_SMD:R_0201_0603Metric"
 			(at 38.862 26.67 90)
 			(effects
@@
 			)
 		)
-		(property "Footprint" ""
+		(property "Footprint" "Capacitor_Tantalum_SMD:CP_EIA-1608-08_AVX-J"
 			(at 41.6052 46.99 0)
 			(effects
@@
 			)
 		)
-		(property "Footprint" ""
+		(property "Footprint" "Capacitor_Tantalum_SMD:CP_EIA-1608-08_AVX-J"
 			(at 183.8452 45.72 0)
 			(effects
@@
 			)
 		)
-		(property "Footprint" ""
+		(property "Footprint" "Package_TO_SOT_SMD:SOT-23"
 			(at 142.24 45.72 0)
 			(effects

Commit message: update
Connections:
- net VDD is gone; now on net +3V3: BZ1.1 (+), D9.1 (K)
Changed lines of the file:
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@@
 			)
 		)
-		(property "Value" "VDD"
+		(property "Value" "+3V3"
 			(at 137.16 16.51 0)
 			(effects

Commit message: update
Parts:
- C24, C25, C26, C27, C28, C29: footprint Capacitor_Tantalum_SMD:CP_EIA-1608-08_AVX-J -> Capacitor_SMD:C_0603_1608Metric
- D10: footprint LED_SMD:LED_0805_2012Metric -> LED_SMD:LED_0603_1608Metric
- R10: value R -> 470k; footprint Resistor_SMD:R_0201_0603Metric -> Resistor_SMD:R_0603_1608Metric
- R11, R12, R8, R9: footprint Resistor_SMD:R_0201_0603Metric -> Resistor_SMD:R_0603_1608Metric
- SW3, SW4, SW5, SW6: footprint Button_Switch_SMD:Nidec_Copal_CAS-120A -> Button_Switch_SMD:SW_SPST_EVQP0
- U4: footprint Display:EA_DOGS104X-A -> Connector_PinHeader_2.54mm:PinHeader_1x04_P2.54mm_Vertical
Changed lines of the file:
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@@
 		(stroke
 			(width 0)
-			(type default)
+			(type dash)
 		)
 		(fill
@@
 		(stroke
 			(width 0)
-			(type default)
+			(type dash)
 		)
 		(fill
@@
 		(stroke
 			(width 0)
-			(type default)
+			(type dash)
 		)
 		(fill
@@
 		(stroke
 			(width 0)
-			(type default)
+			(type dash)
 		)
 		(fill
@@
 			)
 		)
-		(property "Footprint" "LED_SMD:LED_0805_2012Metric"
+		(property "Footprint" "LED_SMD:LED_0603_1608Metric"
 			(at 135.89 86.36 0)
 			(effects
@@
 			)
 		)
-		(property "Footprint" "Resistor_SMD:R_0201_0603Metric"
+		(property "Footprint" "Resistor_SMD:R_0603_1608Metric"
 			(at 87.122 26.67 90)
 			(effects
@@
 			)
 		)
-		(property "Footprint" "Button_Switch_SMD:Nidec_Copal_CAS-120A"
+		(property "Footprint" "Button_Switch_SMD:SW_SPST_EVQP0"
 			(at 58.42 87.63 0)
 			(effects
@@
 			)
 		)
-		(property "Footprint" "Button_Switch_SMD:Nidec_Copal_CAS-120A"
+		(property "Footprint" "Button_Switch_SMD:SW_SPST_EVQP0"
 			(at 106.68 87.63 0)
 			(effects
@@
 			)
 		)
-		(property "Footprint" "Capacitor_Tantalum_SMD:CP_EIA-1608-08_AVX-J"
+		(property "Footprint" "Capacitor_SMD:C_0603_1608Metric"
 			(at 89.8652 93.98 0)
 			(effects
@@
 			)
 		)
-		(property "Value" "R"
+		(property "Value" "470k"
 			(at 91.44 74.9299 0)
 			(effects
@@
 			)
 		)
-		(property "Footprint" "Resistor_SMD:R_0201_0603Metric"
+		(property "Footprint" "Resistor_SMD:R_0603_1608Metric"
 			(at 87.122 73.66 90)
 			(effects
@@
 			)
 		)
-		(property "Footprint" "Resistor_SMD:R_0201_0603Metric"
+		(property "Footprint" "Resistor_SMD:R_0603_1608Metric"
 			(at 38.862 73.66 90)
 			(effects
@@
 			)
 		)
-		(property "Footprint" "Capacitor_Tantalum_SMD:CP_EIA-1608-08_AVX-J"
+		(property "Footprint" "Capacitor_SMD:C_0603_1608Metric"
 			(at 41.6052 93.98 0)
 			(effects
@@
 			)
 		)
-		(property "Footprint" "Button_Switch_SMD:Nidec_Copal_CAS-120A"
+		(property "Footprint" "Button_Switch_SMD:SW_SPST_EVQP0"
 			(at 53.34 41.91 0)
 			(effects
@@
 			)
 		)
-		(property "Footprint" "Display:EA_DOGS104X-A"
+		(property "Footprint" "Connector_PinHeader_2.54mm:PinHeader_1x04_P2.54mm_Vertical"
 			(at 182.626 29.718 0)
 			(effects
@@
 			)
 		)
-		(property "Footprint" "Capacitor_Tantalum_SMD:CP_EIA-1608-08_AVX-J"
+		(property "Footprint" "Capacitor_SMD:C_0603_1608Metric"
 			(at 195.2752 45.72 0)
 			(effects
@@
 			)
 		)
-		(property "Footprint" "Resistor_SMD:R_0201_0603Metric"
+		(property "Footprint" "Resistor_SMD:R_0603_1608Metric"
 			(at 134.112 78.74 90)
 			(effects
@@
 			)
 		)
-		(property "Footprint" "Capacitor_Tantalum_SMD:CP_EIA-1608-08_AVX-J"
+		(property "Footprint" "Capacitor_SMD:C_0603_1608Metric"
 			(at 89.8652 46.99 0)
 			(effects
@@
 			)
 		)
-		(property "Footprint" "Button_Switch_SMD:Nidec_Copal_CAS-120A"
+		(property "Footprint" "Button_Switch_SMD:SW_SPST_EVQP0"
 			(at 101.6 41.91 0)
 			(effects
@@
 			)
 		)
-		(property "Footprint" "Resistor_SMD:R_0201_0603Metric"
+		(property "Footprint" "Resistor_SMD:R_0603_1608Metric"
 			(at 38.862 26.67 90)
 			(effects
@@
 			)
 		)
-		(property "Footprint" "Capacitor_Tantalum_SMD:CP_EIA-1608-08_AVX-J"
+		(property "Footprint" "Capacitor_SMD:C_0603_1608Metric"
 			(at 41.6052 46.99 0)
 			(effects
@@
 			)
 		)
-		(property "Footprint" "Capacitor_Tantalum_SMD:CP_EIA-1608-08_AVX-J"
+		(property "Footprint" "Capacitor_SMD:C_0603_1608Metric"
 			(at 183.8452 45.72 0)
 			(effects

Commit message: update
Parts:
- removed U4: oled_0.96"_128x64px, Connector_PinHeader_2.54mm:PinHeader_1x04_P2.54mm_Vertical, symbol Display_Graphic:EA_DOGS104B-A
- added U4: oled_0.96"_128x64px, Connector_PinHeader_2.54mm:PinHeader_1x04_P2.54mm_Vertical, symbol libs:EA_DOGS104B-A
Connections:
- net +3V3: now also U4.2 (VDD)
- net GND: now also U4.1 (GND)
- net SCL_DISPLAY: now also U4.3 (SCK)
- net SDA_DISPLAY: now also U4.4 (SDA)
Changed lines of the file:
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@@
+	)
+	(symbol
+		(lib_id "libs:EA_DOGS104B-A")
+		(at 220.98 36.83 0)
+		(unit 1)
+		(exclude_from_sim no)
+		(in_bom yes)
+		(on_board yes)
+		(dnp no)
+		(property "Reference" "U4"
+			(at 215.138 20.32 0)
+			(effects
+				(font
+					(size 1.27 1.27)
+				)
+				(justify left)
+			)
+		)
+		(property "Value" "oled_0.96\"_128x64px"
+			(at 212.852 22.86 0)
+			(effects
+				(font
+					(size 1.27 1.27)
+				)
+				(justify left)
+			)
+		)
+		(property "Footprint" "Connector_PinHeader_2.54mm:PinHeader_1x04_P2.54mm_Vertical"
+			(at 182.626 29.718 0)
+			(effects
+				(font
+					(size 1.27 1.27)
+				)
+				(hide yes)
+			)
+		)
+		(property "Datasheet" "http://www.lcd-module.com/fileadmin/eng/pdf/doma/dogs104e.pdf"
+			(at 169.672 11.684 0)
+			(effects
+				(font
+					(size 1.27 1.27)
+				)
+				(hide yes)
+			)
+		)
+		(property "Description" "LCD 4x10 character display blue transmissive background, +3.3V VDD, I2C or SPI"
+			(at 159.512 4.064 0)
+			(effects
+				(font
+					(size 1.27 1.27)
+				)
+				(hide yes)
+			)
+		)
+		(pin "4"
+		)
+		(pin "1"
+		)
+		(pin "3"
+		)
+		(pin "2"
+		)
+		(instances
+			(project ""
+				(path "/13844229-b559-4868-a710-53f590233cb2/84252bff-756a-4e73-bf59-14a8ed329bed"
+					(reference "U4")
+					(unit 1)
+				)
+			)
+		)
 	)
 	(symbol
@@
 					(unit 1)
 				)
-			)
-		)
-	)
-	(symbol
-		(lib_id "Display_Graphic:EA_DOGS104B-A")
-		(at 220.98 36.83 0)
-		(unit 1)
-		(exclude_from_sim no)
-		(in_bom yes)
-		(on_board yes)
-		(dnp no)
-		(fields_autoplaced yes)
-		(property "Reference" "U4"
-			(at 219.71 21.59 0)
-			(effects
-				(font
-					(size 1.27 1.27)
-				)
-				(justify left)
-			)
-		)
-		(property "Value" "oled_0.96\"_128x64px"
-			(at 210.82 25.146 0)
-			(effects
-				(font
-					(size 1.27 1.27)
-				)
-				(justify left)
-			)
-		)
-		(property "Footprint" "Connector_PinHeader_2.54mm:PinHeader_1x04_P2.54mm_Vertical"
-			(at 182.626 29.718 0)
-			(effects
-				(font
-					(size 1.27 1.27)
-				)
-				(hide yes)
-			)
-		)
-		(property "Datasheet" "http://www.lcd-module.com/fileadmin/eng/pdf/doma/dogs104e.pdf"
-			(at 169.672 11.684 0)
-			(effects
-				(font
-					(size 1.27 1.27)
-				)
-				(hide yes)
-			)
-		)
-		(property "Description" "LCD 4x10 character display blue transmissive background, +3.3V VDD, I2C or SPI"
-			(at 159.512 4.064 0)
-			(effects
-				(font
-					(size 1.27 1.27)
-				)
-				(hide yes)
-			)
-		)
-		(pin "1"
-		)
-		(pin "3"
-		)
-		(pin "2"
-		)
-		(pin "4"
-		)
-		(instances
-			(project ""
-				(path "/13844229-b559-4868-a710-53f590233cb2/84252bff-756a-4e73-bf59-14a8ed329bed"
-					(reference "U4")
-					(unit 1)
-				)

Commit message: update
Other:
- title: (none) -> Interfaccia Utente
Changed lines of the file:
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@@
 	(generator_version "9.0")
 	(paper "A4")
+	(title_block
+		(title "Interfaccia Utente")
+	)
 	(rectangle
 		(start 15.24 15.24)
@@
 		(dnp no)
 		(property "Reference" "U4"
-			(at 215.138 20.32 0)
+			(at 218.948 22.098 0)
 			(effects
 				(font
@@
 		)
 		(property "Value" "oled_0.96\"_128x64px"
-			(at 212.852 22.86 0)
-			(effects
-				(font
+			(at 209.804 25.146 0)
+			(effects
+				(font

Commit message: update
Parts:
- SW3, SW4, SW5, SW6: symbol Switch:SW_MEC_5G -> Switch:SW_Push
Connections:
- net GND: now also SW3.2, SW4.2, SW5.2, SW6.2; no longer SW3.3 (B), SW3.4 (B), SW4.3 (B), SW4.4 (B), SW5.3 (B), SW5.4 (B), SW6.3 (B), SW6.4 (B)
- net SW_DOWN: no longer SW6.2 (A)
- net SW_LEFT: no longer SW4.2 (A)
- net SW_RIGHT: no longer SW5.2 (A)
- net SW_UP: no longer SW3.2 (A)
Changed lines of the file:
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@@
 	)
 	(symbol
-		(lib_id "Switch:SW_MEC_5G")
+		(lib_id "Switch:SW_Push")
 		(at 53.34 87.63 270)
 		(unit 1)
@@
 			)
 		)
-		(property "Datasheet" "http://www.apem.com/int/index.php?controller=attachment&id_attachment=488"
+		(property "Datasheet" "~"
 			(at 58.42 87.63 0)
 			(effects
@@
 			)
 		)
-		(property "Description" "MEC 5G single pole normally-open tactile switch"
+		(property "Description" "Push button switch, generic, two pins"
 			(at 53.34 87.63 0)
 			(effects
@@
 		(pin "2"
 		)
-		(pin "4"
-		)
-		(pin "3"
-		)
 		(pin "1"
 		)
@@
 	)
 	(symbol
-		(lib_id "Switch:SW_MEC_5G")
+		(lib_id "Switch:SW_Push")
 		(at 101.6 87.63 270)
 		(unit 1)
@@
 			)
 		)
-		(property "Datasheet" "http://www.apem.com/int/index.php?controller=attachment&id_attachment=488"
+		(property "Datasheet" "~"
 			(at 106.68 87.63 0)
 			(effects
@@
 			)
 		)
-		(property "Description" "MEC 5G single pole normally-open tactile switch"
+		(property "Description" "Push button switch, generic, two pins"
 			(at 101.6 87.63 0)
 			(effects
@@
 		)
 		(pin "2"
-		)
-		(pin "4"
-		)
-		(pin "3"
 		)
 		(pin "1"
@@
 	)
 	(symbol
-		(lib_id "Switch:SW_MEC_5G")
+		(lib_id "Switch:SW_Push")
 		(at 48.26 41.91 270)
 		(unit 1)
@@
 			)
 		)
-		(property "Datasheet" "http://www.apem.com/int/index.php?controller=attachment&id_attachment=488"
+		(property "Datasheet" "~"
 			(at 53.34 41.91 0)
 			(effects
@@
 			)
 		)
-		(property "Description" "MEC 5G single pole normally-open tactile switch"
+		(property "Description" "Push button switch, generic, two pins"
 			(at 48.26 41.91 0)
 			(effects
@@
 		)
 		(pin "2"
-		)
-		(pin "4"
-		)
-		(pin "3"
 		)
 		(pin "1"
@@
 	)
 	(symbol
-		(lib_id "Switch:SW_MEC_5G")
+		(lib_id "Switch:SW_Push")
 		(at 96.52 41.91 270)
 		(unit 1)
@@
 			)
 		)
-		(property "Datasheet" "http://www.apem.com/int/index.php?controller=attachment&id_attachment=488"
+		(property "Datasheet" "~"
 			(at 101.6 41.91 0)
 			(effects
@@
 			)
 		)
-		(property "Description" "MEC 5G single pole normally-open tactile switch"
+		(property "Description" "Push button switch, generic, two pins"
 			(at 96.52 41.91 0)
 			(effects
@@
 		(pin "2"
 		)
-		(pin "4"
-		)
-		(pin "3"
-		)
-		(pin "1"
+		(pin "1"
